File: kicad/DTE - Atlys VHDCI.sch (KiCad schematic (older format))
At the start: 3 parts

Commit message: Netlist DRC pass - fixed pins types, incorrect connections, added PWRFLAGS
Parts:
- gave numbers to parts that had none: 3
Connections:
- net GND: now also J201.36 (GND), J201.39 (GND), J201.42 (GND), J201.45 (GND), J201.48 (GND), J201.55 (GND), J201.58 (GND), J201.61 (GND), J201.64 (GND), J201.67 (GND)
Changed lines of the file:
@@
 $EndDescr
 $Comp
-L R R?
+L R R201
 U 1 1 53A5882A
 P 4450 5750
-F 0 "R?" V 4530 5750 40  0000 C CNN
+F 0 "R201" V 4530 5750 40  0000 C CNN
 F 1 "1M" V 4457 5751 40  0000 C CNN
 F 2 "~" V 4380 5750 30  0000 C CNN
@@
 $EndComp
 $Comp
-L C C?
+L C C201
 U 1 1 53A58839
 P 4450 6050
-F 0 "C?" H 4450 6150 40  0000 L CNN
-F 1 "1n" H 4456 5965 40  0000 L CNN
+F 0 "C201" V 4500 5820 40  0000 L CNN
+F 1 "1n" V 4400 5900 40  0000 L CNN
 F 2 "~" H 4488 5900 30  0000 C CNN
 F 3 "~" H 4450 6050 60  0000 C CNN
@@
 Text HLabel 3650 1700 0    60   Output ~ 0
 5V
-Text HLabel 3650 1850 0    60   Output ~ 0
+Text HLabel 3650 1800 0    60   Output ~ 0
 VCC
 Text HLabel 4450 4450 0    60   Output ~ 0
@@
 RTS4
 $Comp
-L DIGILENT_VHDCI_CONN J?
+L DIGILENT_VHDCI_CONN J201
 U 1 1 53A5DC31
 P 5850 3950
-F 0 "J?" H 5500 1950 60  0000 C CNN
+F 0 "J201" H 5550 1950 60  0000 C CNN
 F 1 "DIGILENT_VHDCI_CONN" H 5450 5850 60  0000 L CNN
 F 2 "~" H 5450 5650 60  0000 C CNN
@@
 	5150 2350 5000 2350
 Wire Wire Line
-	5000 2350 5000 2650
-Wire Wire Line
-	5000 2650 5000 2950
-Wire Wire Line
-	5000 2950 5000 3250
-Wire Wire Line
-	5000 3250 5000 3550
-Wire Wire Line
-	5000 3550 5000 4250
-Wire Wire Line
-	5000 4250 5000 4550
-Wire Wire Line
-	5000 4550 5000 4850
-Wire Wire Line
-	5000 4850 5000 5150
-Wire Wire Line
-	5000 5150 5000 5450
-Wire Wire Line
-	3750 5450 5000 5450
-Wire Wire Line
-	5000 5450 5150 5450
+	5000 1900 5000 5450
+Wire Wire Line
+	3750 5450 5150 5450
 Wire Wire Line
 	5150 5150 5000 5150
@@
 	6800 5450 6600 5450
 Wire Wire Line
-	6800 2350 6800 2650
-Wire Wire Line
-	6800 2650 6800 2950
-Wire Wire Line
-	6800 2950 6800 3250
-Wire Wire Line
-	6800 3250 6800 3550
-Wire Wire Line
-	6800 3550 6800 4250
-Wire Wire Line
-	6800 4250 6800 4550
-Wire Wire Line
-	6800 4550 6800 4850
-Wire Wire Line
-	6800 4850 6800 5150
-Wire Wire Line
-	6800 5150 6800 5450
+	6800 1900 6800 5450
 Wire Wire Line
 	6800 2350 6600 2350
@@
 	6600 2650 6800 2650
 Connection ~ 6800 2650
-Wire Wire Line
-	6600 2950 6800 2950
 Connection ~ 6800 2950
 Wire Wire Line
@@
 	6800 5750 6600 5750
 Wire Wire Line
-	4700 5750 5000 5750
-Wire Wire Line
-	5000 5750 5150 5750
+	4700 5750 5150 5750
 Wire Wire Line
 	5000 5750 5000 6050
 Wire Wire Line
-	4650 6050 5000 6050
-Wire Wire Line
-	5000 6050 6800 6050
+	4650 6050 6800 6050
 Wire Wire Line
 	6600 5550 7350 5550
@@
 Connection ~ 5000 6050
 Wire Wire Line
-	3500 6050 3750 6050
-Wire Wire Line
-	3750 6050 4250 6050
+	3500 6050 4250 6050
 Wire Wire Line
 	4200 5750 3750 5750
@@
 Connection ~ 6900 3750
 Wire Wire Line
-	6900 1850 6900 3750
-Wire Wire Line
-	6900 3750 6900 4050
-Wire Wire Line
-	3650 1850 4900 1850
-Wire Wire Line
-	4900 1850 6900 1850
-Connection ~ 4900 1850
+	6900 1800 6900 4050
+Wire Wire Line
+	3650 1800 6900 1800
+Connection ~ 4900 1800
 Connection ~ 4800 3850
 Wire Wire Line
-	3650 1700 4800 1700
-Wire Wire Line
-	4800 1700 7000 1700
-Wire Wire Line
-	7000 1700 7000 3850
-Wire Wire Line
-	7000 3850 7000 3950
+	3650 1700 7000 1700
+Wire Wire Line
+	7000 1700 7000 3950
 Connection ~ 7000 3850
 Connection ~ 4800 1700
@@
 	6600 4150 7350 4150
 Wire Wire Line
-	4800 1700 4800 3850
-Wire Wire Line
-	4800 3850 4800 3950
-Wire Wire Line
-	4900 1850 4900 3750
-Wire Wire Line
-	4900 3750 4900 4050
-Wire Wire Line
-	3750 5450 3750 5750
-Wire Wire Line
-	3750 5750 3750 6050
+	4800 1700 4800 3950
+Wire Wire Line
+	4900 1800 4900 4050
+Wire Wire Line
+	3750 5450 3750 6050
 Connection ~ 3750 6050
+$Comp
+L PWR_FLAG #FLG201
+U 1 1 53C07D98
+P 3750 5450
+F 0 "#FLG201" H 3750 5545 30  0001 C CNN
+F 1 "PWR_FLAG" H 3750 5630 30  0001 C CNN
+F 2 "" H 3750 5450 60  0000 C CNN
+F 3 "" H 3750 5450 60  0000 C CNN
+	1    3750 5450
+	1    0    0    -1
+$EndComp
+Wire Wire Line
+	6600 2950 6800 2950
+Wire Wire Line
+	6800 1900 5000 1900
+Connection ~ 5000 2350
+Connection ~ 6800 2350
 $EndSCHEMATC

Commit message: Updated notes and sheet names
Other:
- note added: "VHDCI connector gives access to FPGA pins on Digilent Atlys FPGA development board"
Changed lines of the file:
@@
 Date "23 jun 2014"
 Rev ""
-Comp ""
+Comp "TimVideos"
 Comment1 ""
 Comment2 ""
@@
 Connection ~ 5000 2350
 Connection ~ 6800 2350
+Text Notes 1900 7250 0    60   ~ 0
+VHDCI connector gives access to FPGA pins on Digilent Atlys FPGA development board
 $EndSCHEMATC
