File: kicad/DTE - PIC18 USB.sch (KiCad schematic (older format))
At the start: 2 parts

Commit message: ID detection changed from RC to EEPROM based, D.board pinout changed, PIC18F85J94 added
Parts:
- added U?: PIC18F85J94, ~, symbol PIC18F85J94
Changed lines of the file:
@@
 LIBS:si8660
 LIBS:pic16f1704
+LIBS:PIC18F85J94
+LIBS:24AA014
 LIBS:Main-cache
 EELAYER 27 0
@@
 $Descr A4 11693 8268
 encoding utf-8
-Sheet 3 8
+Sheet 3 7
 Title ""
-Date "22 jun 2014"
+Date "23 jun 2014"
 Rev ""
 Comp ""
@@
 Text HLabel 2250 1300 2    60   BiDi ~ 0
 SCL
+$Comp
+L PIC18F85J94 U?
+U 1 1 53B3C345
+P 3850 4050
+F 0 "U?" H 3450 1600 60  0000 L CNN
+F 1 "PIC18F85J94" H 3450 6550 60  0000 L CNN
+F 2 "~" H 3850 4050 60  0000 C CNN
+F 3 "~" H 3850 4050 60  0000 C CNN
+	1    3850 4050
+	1    0    0    -1
+$EndComp
 $EndSCHEMATC

Commit message: Completed PIC 18 USB sheet; Motherboard schematic done
Parts:
- removed P?: ICSP, symbol CONN_6
- added C?: 4.7n, ~, symbol C
- added C?: CSMALL, ~, symbol CSMALL
- added C? (x5): 0.1u, ~, symbol CSMALL
- added C?: 10u, ~, symbol CSMALL
- added P?: ICSP, symbol CONN_5
- added R?: 10K, ~, symbol R
- added R?: 1M, ~, symbol R
- added U?: AAT3221IGV-3.3-T1, ~, symbol AAT3221IGV-3.3-T1
Connections:
- net labels added: PGC, PGD
- wire segments 0 -> 101
- no-connect marks 0 -> 26
Other:
- moved on the sheet: J?

Commit message: Netlist DRC pass - fixed pins types, incorrect connections, added PWRFLAGS
Parts:
- added R302, R303: 50, ~, symbol R
- added R305: 0.47, ~, symbol R
- added R306: 0.10, ~, symbol R
- gave numbers to parts that had none: 14
Connections:
- wire segments 101 -> 104
Other:
- moved on the sheet: C307, J301, R304, U302
Changed lines of the file:
@@
 $EndDescr
 $Comp
-L USB J?
+L USB J301
 U 1 1 53A79C0D
-P 5700 1650
-F 0 "J?" H 5650 2050 60  0000 C CNN
-F 1 "USB" V 5450 1800 60  0000 C CNN
-F 2 "" H 5700 1650 60  0000 C CNN
-F 3 "" H 5700 1650 60  0000 C CNN
-	1    5700 1650
+P 6400 1650
+F 0 "J301" H 6350 2050 60  0000 C CNN
+F 1 "USB" V 6150 1800 60  0000 C CNN
+F 2 "" H 6400 1650 60  0000 C CNN
+F 3 "" H 6400 1650 60  0000 C CNN
+	1    6400 1650
 	-1   0    0    -1
 $EndComp
@@
 SCL
 $Comp
-L PIC18F85J94 U?
+L PIC18F85J94 U301
 U 1 1 53B3C345
 P 3850 4050
-F 0 "U?" H 3450 1600 60  0000 L CNN
+F 0 "U301" H 3450 1600 60  0000 L CNN
 F 1 "PIC18F85J94" H 3450 6550 60  0000 L CNN
 F 2 "~" H 3850 4050 60  0000 C CNN
@@
 $EndComp
 $Comp
-L R R?
+L R R301
 U 1 1 53B87E95
 P 2700 6250
-F 0 "R?" V 2780 6250 40  0000 C CNN
+F 0 "R301" V 2780 6250 40  0000 C CNN
 F 1 "10K" V 2707 6251 40  0000 C CNN
 F 2 "~" V 2630 6250 30  0000 C CNN
@@
 $EndComp
 $Comp
-L AAT3221IGV-3.3-T1 U?
+L AAT3221IGV-3.3-T1 U302
 U 1 1 53BF3199
-P 7700 2050
-F 0 "U?" H 7500 1700 60  0000 L CNN
-F 1 "AAT3221IGV-3.3-T1" H 7700 2400 60  0000 C CNN
-F 2 "~" H 7750 2150 60  0000 C CNN
-F 3 "~" H 7750 2150 60  0000 C CNN
-	1    7700 2050
-	1    0    0    -1
-$EndComp
-$Comp
-L R R?
+P 8400 2050
+F 0 "U302" H 8200 1700 60  0000 L CNN
+F 1 "AAT3221IGV-3.3-T1" H 8400 2400 60  0000 C CNN
+F 2 "~" H 8450 2150 60  0000 C CNN
+F 3 "~" H 8450 2150 60  0000 C CNN
+	1    8400 2050
+	1    0    0    -1
+$EndComp
+$Comp
+L R R304
 U 1 1 53BF3289
-P 6100 2850
-F 0 "R?" V 6180 2850 40  0000 C CNN
-F 1 "1M" V 6107 2851 40  0000 C CNN
-F 2 "~" V 6030 2850 30  0000 C CNN
-F 3 "~" H 6100 2850 30  0000 C CNN
-	1    6100 2850
-	1    0    0    -1
-$EndComp
-$Comp
-L C C?
+P 6800 2850
+F 0 "R304" V 6880 2850 40  0000 C CNN
+F 1 "1M" V 6807 2851 40  0000 C CNN
+F 2 "~" V 6730 2850 30  0000 C CNN
+F 3 "~" H 6800 2850 30  0000 C CNN
+	1    6800 2850
+	1    0    0    -1
+$EndComp
+$Comp
+L C C307
 U 1 1 53BF32B6
-P 6400 2850
-F 0 "C?" H 6400 2950 40  0000 L CNN
-F 1 "4.7n" H 6406 2765 40  0000 L CNN
-F 2 "~" H 6438 2700 30  0000 C CNN
-F 3 "~" H 6400 2850 60  0000 C CNN
-	1    6400 2850
-	1    0    0    -1
-$EndComp
-$Comp
-L CONN_5 P?
+P 7100 2850
+F 0 "C307" H 7100 2950 40  0000 L CNN
+F 1 "4.7n" H 7106 2765 40  0000 L CNN
+F 2 "~" H 7138 2700 30  0000 C CNN
+F 3 "~" H 7100 2850 60  0000 C CNN
+	1    7100 2850
+	1    0    0    -1
+$EndComp
+$Comp
+L CONN_5 P301
 U 1 1 53BF41FB
 P 2850 7200
-F 0 "P?" V 2800 7200 50  0000 C CNN
+F 0 "P301" V 2800 7200 50  0000 C CNN
 F 1 "ICSP" V 2900 7200 50  0000 C CNN
 F 2 "" H 2850 7200 60  0000 C CNN
@@
 $EndComp
 $Comp
-L CSMALL C?
+L CSMALL C308
 U 1 1 53BFC72A
-P 8450 2300
-F 0 "C?" H 8475 2350 30  0000 L CNN
-F 1 "CSMALL" H 8475 2250 30  0000 L CNN
-F 2 "~" H 8450 2300 60  0000 C CNN
-F 3 "~" H 8450 2300 60  0000 C CNN
-	1    8450 2300
+P 9500 2450
+F 0 "C308" H 9525 2500 30  0000 L CNN
+F 1 "CSMALL" H 9525 2400 30  0000 L CNN
+F 2 "~" H 9500 2450 60  0000 C CNN
+F 3 "~" H 9500 2450 60  0000 C CNN
+	1    9500 2450
 	1    0    0    -1
 $EndComp
@@
 	2950 6250 3150 6250
 Wire Wire Line
-	6100 1850 7200 1850
-Wire Wire Line
-	7000 1850 7000 1850
-Wire Wire Line
-	7000 1850 7000 2250
-Connection ~ 7000 1850
-Wire Wire Line
-	6100 2000 6300 2000
-Wire Wire Line
-	6300 2000 6400 2050
-Wire Wire Line
-	6400 2050 7200 2050
-Wire Wire Line
-	5350 2100 5200 2100
-Wire Wire Line
-	5200 2100 5200 2400
-Wire Wire Line
-	5200 2400 6250 2400
-Wire Wire Line
-	6250 2100 6250 2550
-Wire Wire Line
-	6250 2100 6100 2100
-Wire Wire Line
-	6100 2600 6100 2550
-Wire Wire Line
-	6100 2550 6400 2550
-Wire Wire Line
-	6400 2550 6400 2650
-Wire Wire Line
-	6400 3050 6400 3150
-Wire Wire Line
-	6100 3150 6100 3100
-Connection ~ 6250 2550
-Connection ~ 6250 2400
-Connection ~ 6800 2050
-Connection ~ 6800 3150
-Wire Wire Line
-	7000 2250 7200 2250
-Wire Wire Line
-	8200 1850 8450 1850
-Wire Wire Line
-	6100 3150 8450 3150
-Connection ~ 6400 3150
-Wire Wire Line
-	5350 1850 5000 1850
+	7450 1850 7900 1850
+Wire Wire Line
+	7700 1850 7700 2250
+Connection ~ 7700 1850
+Wire Wire Line
+	6800 2000 7000 2000
+Wire Wire Line
+	7000 2000 7100 2050
+Wire Wire Line
+	7100 2050 7900 2050
+Wire Wire Line
+	6050 2100 5900 2100
+Wire Wire Line
+	5900 2100 5900 2400
+Wire Wire Line
+	5900 2400 6950 2400
+Wire Wire Line
+	6950 2100 6950 2550
+Wire Wire Line
+	6950 2100 6800 2100
+Wire Wire Line
+	6800 2600 6800 2550
+Wire Wire Line
+	6800 2550 7100 2550
+Wire Wire Line
+	7100 2550 7100 2650
+Wire Wire Line
+	7100 3050 7100 3150
+Wire Wire Line
+	6800 3150 6800 3100
+Connection ~ 6950 2550
+Connection ~ 6950 2400
+Connection ~ 7500 2050
+Connection ~ 7500 3150
+Wire Wire Line
+	7700 2250 7900 2250
+Wire Wire Line
+	6800 3150 9500 3150
+Connection ~ 7100 3150
 Wire Wire Line
 	5000 1850 4900 1950
@@
 Wire Wire Line
 	4900 1850 5050 2000
-Wire Wire Line
-	5050 2000 5350 2000
 Wire Wire Line
 	2550 3950 3150 3950
@@
 Connection ~ 3050 6250
 Wire Wire Line
-	8450 1850 8450 2200
-Connection ~ 8450 1850
+	9500 1850 9500 2350
+Connection ~ 9500 1850
 Text Label 7650 5550 2    60   ~ 0
 GND
@@
 	6350 5050 4600 5050
 $Comp
-L CSMALL C?
+L CSMALL C304
 U 1 1 53BFC8D3
 P 5600 5300
-F 0 "C?" H 5625 5350 30  0000 L CNN
+F 0 "C304" H 5625 5350 30  0000 L CNN
 F 1 "0.1u" H 5625 5250 30  0000 L CNN
 F 2 "~" H 5600 5300 60  0000 C CNN
@@
 $EndComp
 $Comp
-L CSMALL C?
+L CSMALL C305
 U 1 1 53BFC8EF
 P 5750 5300
-F 0 "C?" H 5775 5350 30  0000 L CNN
+F 0 "C305" H 5775 5350 30  0000 L CNN
 F 1 "0.1u" H 5775 5250 30  0000 L CNN
 F 2 "~" H 5750 5300 60  0000 C CNN
@@
 $EndComp
 $Comp
-L CSMALL C?
+L CSMALL C306
 U 1 1 53BFC8F5
 P 5900 5300
-F 0 "C?" H 5925 5350 30  0000 L CNN
+F 0 "C306" H 5925 5350 30  0000 L CNN
 F 1 "0.1u" H 5925 5250 30  0000 L CNN
 F 2 "~" H 5900 5300 60  0000 C CNN
@@
 Wire Wire Line
 	2450 6250 2350 6250
-Text Label 8450 1850 0    60   ~ 0
-VCC
-Wire Wire Line
-	8450 3150 8450 2400
-Text Label 6800 3150 0    60   ~ 0
+Text Label 9500 1850 0    60   ~ 0
+VCC
+Text Label 7500 3150 0    60   ~ 0
 GND
-Text Label 7000 1850 0    60   ~ 0
+Text Label 7700 1850 0    60   ~ 0
 5V
 Wire Wire Line
-	6800 3150 6800 2050
+	7500 3150 7500 2050
 Wire Wire Line
 	5600 5200 5600 4850
@@
 	5350 5250 5350 5400
 $Comp
-L CSMALL C?
+L CSMALL C303
 U 1 1 53BFCFE3
 P 5350 5500
-F 0 "C?" H 5375 5550 30  0000 L CNN
+F 0 "C303" H 5375 5550 30  0000 L CNN
 F 1 "10u" H 5375 5450 30  0000 L CNN
 F 2 "~" H 5350 5500 60  0000 C CNN
@@
 Connection ~ 5350 5750
 $Comp
-L CSMALL C?
+L CSMALL C302
 U 1 1 53BFD04A
 P 5050 5550
-F 0 "C?" H 5075 5600 30  0000 L CNN
+F 0 "C302" H 5075 5600 30  0000 L CNN
 F 1 "0.1u" H 5075 5500 30  0000 L CNN
 F 2 "~" H 5050 5550 60  0000 C CNN
@@
 	4900 5400 4900 5450
 $Comp
-L CSMALL C?
+L CSMALL C301
 U 1 1 53BFD2B0
 P 4900 5550
-F 0 "C?" H 4925 5600 30  0000 L CNN
+F 0 "C301" H 4925 5600 30  0000 L CNN
 F 1 "0.1u" H 4925 5500 30  0000 L CNN
 F 2 "~" H 4900 5550 60  0000 C CNN
@@
 NoConn ~ 4600 4650
 NoConn ~ 4600 1750
+$Comp
+L R R302
+U 1 1 53C0EA4A
+P 5450 1850
+F 0 "R302" V 5500 1600 40  0000 C CNN
+F 1 "50" V 5457 1851 40  0000 C CNN
+F 2 "~" V 5380 1850 30  0000 C CNN
+F 3 "~" H 5450 1850 30  0000 C CNN
+	1    5450 1850
+	0    -1   -1   0
+$EndComp
+$Comp
+L R R303
+U 1 1 53C0EA59
+P 5450 2000
+F 0 "R303" V 5500 1750 40  0000 C CNN
+F 1 "50" V 5457 2001 40  0000 C CNN
+F 2 "~" V 5380 2000 30  0000 C CNN
+F 3 "~" H 5450 2000 30  0000 C CNN
+	1    5450 2000
+	0    -1   -1   0
+$EndComp
+Wire Wire Line
+	5200 1850 5000 1850
+Wire Wire Line
+	5700 1850 6050 1850
+Wire Wire Line
+	5050 2000 5200 2000
+Wire Wire Line
+	5700 2000 6050 2000
+$Comp
+L R R305
+U 1 1 53C0ECE1
+P 7200 1850
+F 0 "R305" V 7280 1850 40  0000 C CNN
+F 1 "0.47" V 7207 1851 40  0000 C CNN
+F 2 "~" V 7130 1850 30  0000 C CNN
+F 3 "~" H 7200 1850 30  0000 C CNN
+	1    7200 1850
+	0    -1   -1   0
+$EndComp
+Wire Wire Line
+	6950 1850 6800 1850
+Wire Wire Line
+	9500 3150 9500 2550
+$Comp
+L R R306
+U 1 1 53C0F13C
+P 9200 1850
+F 0 "R306" V 9280 1850 40  0000 C CNN
+F 1 "0.10" V 9207 1851 40  0000 C CNN
+F 2 "~" V 9130 1850 30  0000 C CNN
+F 3 "~" H 9200 1850 30  0000 C CNN
+	1    9200 1850
+	0    -1   -1   0
+$EndComp
+Wire Wire Line
+	8950 1850 8900 1850
+Wire Wire Line
+	9450 1850 9500 1850
+Text Label 5900 5750 0    60   ~ 0
+GND
 $EndSCHEMATC

Commit message: Updated notes and sheet names
Other:
- note added: "PIC18F85J94 MCU simulates production board for HDMI2USB as well as enables standalone operation using USB interface."
- moved on the sheet: C307, J301, P301, R301, R302, R303, R304, R305, R306, U301, U302

Commit message: Fixed Csmall not showing up in some versions of kicad. Fixed C308
Parts:
- C308: value CSMALL -> 0.1u
Changed lines of the file:
@@
 LIBS:AAT3221IGV-3V3-T1
 LIBS:CONN_16
+LIBS:csmall
 LIBS:Motherboard-cache
 EELAYER 27 0
@@
 	0    1    1    0
 $EndComp
-$Comp
-L CSMALL C308
-U 1 1 53BFC72A
-P 9400 2200
-F 0 "C308" H 9425 2250 30  0000 L CNN
-F 1 "CSMALL" H 9425 2150 30  0000 L CNN
-F 2 "~" H 9400 2200 60  0000 C CNN
-F 3 "~" H 9400 2200 60  0000 C CNN
-	1    9400 2200
-	1    0    0    -1
-$EndComp
 Wire Wire Line
 	2850 6000 3050 6000
@@
 Wire Wire Line
 	6250 4800 4500 4800
-$Comp
-L CSMALL C304
-U 1 1 53BFC8D3
-P 5500 5050
-F 0 "C304" H 5525 5100 30  0000 L CNN
-F 1 "0.1u" H 5525 5000 30  0000 L CNN
-F 2 "~" H 5500 5050 60  0000 C CNN
-F 3 "~" H 5500 5050 60  0000 C CNN
-	1    5500 5050
-	1    0    0    -1
-$EndComp
-$Comp
-L CSMALL C305
-U 1 1 53BFC8EF
-P 5650 5050
-F 0 "C305" H 5675 5100 30  0000 L CNN
-F 1 "0.1u" H 5675 5000 30  0000 L CNN
-F 2 "~" H 5650 5050 60  0000 C CNN
-F 3 "~" H 5650 5050 60  0000 C CNN
-	1    5650 5050
-	1    0    0    -1
-$EndComp
-$Comp
-L CSMALL C306
-U 1 1 53BFC8F5
-P 5800 5050
-F 0 "C306" H 5825 5100 30  0000 L CNN
-F 1 "0.1u" H 5825 5000 30  0000 L CNN
-F 2 "~" H 5800 5050 60  0000 C CNN
-F 3 "~" H 5800 5050 60  0000 C CNN
-	1    5800 5050
-	1    0    0    -1
-$EndComp
 Wire Wire Line
 	6250 4600 6250 4800
@@
 Wire Wire Line
 	5250 5000 5250 5150
-$Comp
-L CSMALL C303
-U 1 1 53BFCFE3
-P 5250 5250
-F 0 "C303" H 5275 5300 30  0000 L CNN
-F 1 "10u" H 5275 5200 30  0000 L CNN
-F 2 "~" H 5250 5250 60  0000 C CNN
-F 3 "~" H 5250 5250 60  0000 C CNN
-	1    5250 5250
-	1    0    0    -1
-$EndComp
 Wire Wire Line
 	5250 5350 5250 5500
 Connection ~ 5250 5500
-$Comp
-L CSMALL C302
-U 1 1 53BFD04A
-P 4950 5300
-F 0 "C302" H 4975 5350 30  0000 L CNN
-F 1 "0.1u" H 4975 5250 30  0000 L CNN
-F 2 "~" H 4950 5300 60  0000 C CNN
-F 3 "~" H 4950 5300 60  0000 C CNN
-	1    4950 5300
-	1    0    0    -1
-$EndComp
 Wire Wire Line
 	4500 5100 4950 5100
@@
 Wire Wire Line
 	4800 5150 4800 5200
-$Comp
-L CSMALL C301
-U 1 1 53BFD2B0
-P 4800 5300
-F 0 "C301" H 4825 5350 30  0000 L CNN
-F 1 "0.1u" H 4825 5250 30  0000 L CNN
-F 2 "~" H 4800 5300 60  0000 C CNN
-F 3 "~" H 4800 5300 60  0000 C CNN
-	1    4800 5300
-	1    0    0    -1
-$EndComp
 Wire Wire Line
 	4800 5400 4800 5500
@@
 Text Notes 700  7600 0    60   ~ 0
 PIC18F85J94 MCU simulates production board for HDMI2USB as well as enables standalone operation using USB interface.
+$Comp
+L CSMALL C308
+U 1 1 53A91209
+P 9400 2200
+F 0 "C308" H 9425 2250 30  0000 L CNN
+F 1 "0.1u" H 9425 2150 30  0000 L CNN
+F 2 "~" H 9400 2200 60  0000 C CNN
+F 3 "~" H 9400 2200 60  0000 C CNN
+	1    9400 2200
+	1    0    0    -1
+$EndComp
+$Comp
+L CSMALL C301
+U 1 1 53A91222
+P 4800 5300
+F 0 "C301" H 4825 5350 30  0000 L CNN
+F 1 "0.1u" H 4825 5250 30  0000 L CNN
+F 2 "~" H 4800 5300 60  0000 C CNN
+F 3 "~" H 4800 5300 60  0000 C CNN
+	1    4800 5300
+	1    0    0    -1
+$EndComp
+$Comp
+L CSMALL C302
+U 1 1 53A9123B
+P 4950 5300
+F 0 "C302" H 4975 5350 30  0000 L CNN
+F 1 "0.1u" H 4975 5250 30  0000 L CNN
+F 2 "~" H 4950 5300 60  0000 C CNN
+F 3 "~" H 4950 5300 60  0000 C CNN
+	1    4950 5300
+	1    0    0    -1
+$EndComp
+$Comp
+L CSMALL C303
+U 1 1 53A91254
+P 5250 5250
+F 0 "C303" H 5275 5300 30  0000 L CNN
+F 1 "10u" H 5275 5200 30  0000 L CNN
+F 2 "~" H 5250 5250 60  0000 C CNN
+F 3 "~" H 5250 5250 60  0000 C CNN
+	1    5250 5250
+	1    0    0    -1
+$EndComp
+$Comp
+L CSMALL C304
+U 1 1 53A9126D
+P 5500 5050
+F 0 "C304" H 5525 5100 30  0000 L CNN
+F 1 "0.1u" H 5525 5000 30  0000 L CNN
+F 2 "~" H 5500 5050 60  0000 C CNN
+F 3 "~" H 5500 5050 60  0000 C CNN
+	1    5500 5050
+	1    0    0    -1
+$EndComp
+$Comp
+L CSMALL C305
+U 1 1 53A91286
+P 5650 5050
+F 0 "C305" H 5675 5100 30  0000 L CNN
+F 1 "0.1u" H 5675 5000 30  0000 L CNN
+F 2 "~" H 5650 5050 60  0000 C CNN
+F 3 "~" H 5650 5050 60  0000 C CNN
+	1    5650 5050
+	1    0    0    -1
+$EndComp
+$Comp
+L CSMALL C306
+U 1 1 53A9129F
+P 5800 5050
+F 0 "C306" H 5825 5100 30  0000 L CNN
+F 1 "0.1u" H 5825 5000 30  0000 L CNN
+F 2 "~" H 5800 5050 60  0000 C CNN
+F 3 "~" H 5800 5050 60  0000 C CNN
+	1    5800 5050
+	1    0    0    -1
+$EndComp
 $EndSCHEMATC
