File: kicad/DTE - PIC18 USB.sch (KiCad schematic (older format))
At the start: 18 parts, among them J301 USB, P301 ICSP, U301 PIC18F85J94, U302 AAT3221IGV-3.3-T1

Commit message: Removed ID controller.sch
Connections:
- wire segments 104 -> 123
Changed lines of the file:
@@
 $EndComp
 Wire Wire Line
-	2850 6000 3050 6000
-Wire Wire Line
-	7350 1600 7800 1600
+	2850 6000 2950 6000
+Wire Wire Line
+	2950 6000 3050 6000
+Wire Wire Line
+	7350 1600 7600 1600
+Wire Wire Line
+	7600 1600 7800 1600
 Wire Wire Line
 	7600 1600 7600 2000
@@
 	6900 1750 7000 1800
 Wire Wire Line
-	7000 1800 7800 1800
+	7000 1800 7400 1800
+Wire Wire Line
+	7400 1800 7800 1800
 Wire Wire Line
 	5950 1850 5800 1850
@@
 	5800 2150 6850 2150
 Wire Wire Line
-	6850 1850 6850 2300
+	6850 1850 6850 2150
+Wire Wire Line
+	6850 2150 6850 2300
 Wire Wire Line
 	6850 1850 6700 1850
@@
 	6700 2350 6700 2300
 Wire Wire Line
-	6700 2300 7000 2300
+	6700 2300 6850 2300
+Wire Wire Line
+	6850 2300 7000 2300
 Wire Wire Line
 	7000 2300 7000 2400
@@
 	7600 2000 7800 2000
 Wire Wire Line
-	6700 2900 9400 2900
+	6700 2900 7000 2900
+Wire Wire Line
+	7000 2900 7400 2900
+Wire Wire Line
+	7400 2900 9400 2900
 Connection ~ 7000 2900
 Wire Wire Line
@@
 	2850 6400 2850 6550
 Wire Wire Line
-	4500 4600 6250 4600
-Wire Wire Line
-	4500 4700 6250 4700
-Wire Wire Line
-	6250 4800 4500 4800
-Wire Wire Line
-	6250 4600 6250 4800
-Connection ~ 6250 4700
-Connection ~ 6250 4600
-Text Label 6250 4600 0    60   ~ 0
+	5800 4800 5650 4800
+Wire Wire Line
+	5500 4800 4500 4800
+Text Label 5800 4600 0    60   ~ 0
 VCC
 Text Label 2750 6400 1    60   ~ 0
@@
 	7400 2900 7400 1800
 Wire Wire Line
-	5500 4950 5500 4600
-Connection ~ 5500 4600
-Wire Wire Line
-	5650 4950 5650 4700
-Connection ~ 5650 4700
-Wire Wire Line
-	5800 4950 5800 4800
+	5500 4950 5500 4800
+Wire Wire Line
+	5650 4950 5650 4800
+Wire Wire Line
+	5800 4600 5800 4700
+Wire Wire Line
+	5800 4700 5800 4800
+Wire Wire Line
+	5800 4800 5800 4950
 Connection ~ 5800 4800
 Wire Wire Line
-	4500 5500 4500 6000
+	4500 5500 4500 5600
+Wire Wire Line
+	4500 5600 4500 5700
+Wire Wire Line
+	4500 5700 4500 5800
+Wire Wire Line
+	4500 5800 4500 6000
 Connection ~ 4500 5600
 Connection ~ 4500 5700
 Wire Wire Line
-	4500 5500 5800 5500
+	4500 5500 4800 5500
+Wire Wire Line
+	4800 5500 4950 5500
+Wire Wire Line
+	4950 5500 5250 5500
+Wire Wire Line
+	5250 5500 5500 5500
+Wire Wire Line
+	5500 5500 5650 5500
+Wire Wire Line
+	5650 5500 5800 5500
 Wire Wire Line
 	5800 5500 5800 5150
@@
 	1    0    0    -1
 $EndComp
+Connection ~ 5800 4700
+Connection ~ 5800 4600
+Wire Wire Line
+	4500 4700 5800 4700
+Wire Wire Line
+	4500 4600 5500 4600
+Wire Wire Line
+	5500 4600 5800 4600
+Connection ~ 5650 4800
+Connection ~ 5500 4800
+Wire Wire Line
+	5650 4800 5500 4800
 $EndSCHEMATC

Commit message: fixed untracked files
Parts:
- added D? (x8): LED, ~, symbol LED
- added P?: UART2, symbol CONN_2
- added R? (x8): 330, ~, symbol R
Connections:
- wire segments 123 -> 158
- no-connect marks 26 -> 16

Commit message: Changed UART debug connector from 2 pin to 4 pin and annotated unannotated parts
Parts:
- removed P?: UART2, symbol CONN_2
- added P302: UART2, symbol CONN_4
- gave numbers to parts that had none: 16
Connections:
- wire segments 158 -> 156
Changed lines of the file:
@@
 $EndComp
 $Comp
-L LED D?
+L LED D308
 U 1 1 53A903F4
 P 6250 3800
-F 0 "D?" H 6235 3870 24  0000 C CNN
+F 0 "D308" H 6235 3870 24  0000 C CNN
 F 1 "LED" H 6250 3700 50  0001 C CNN
 F 2 "~" H 6250 3800 60  0000 C CNN
@@
 $EndComp
 $Comp
-L LED D?
+L LED D307
 U 1 1 53A90444
 P 6100 3800
-F 0 "D?" H 6085 3870 24  0000 C CNN
+F 0 "D307" H 6085 3870 24  0000 C CNN
 F 1 "LED" H 6100 3700 50  0001 C CNN
 F 2 "~" H 6100 3800 60  0000 C CNN
@@
 $EndComp
 $Comp
-L LED D?
+L LED D306
 U 1 1 53A9044A
 P 5950 3800
-F 0 "D?" H 5935 3870 24  0000 C CNN
+F 0 "D306" H 5935 3870 24  0000 C CNN
 F 1 "LED" H 5950 3700 50  0001 C CNN
 F 2 "~" H 5950 3800 60  0000 C CNN
@@
 $EndComp
 $Comp
-L LED D?
+L LED D305
 U 1 1 53A90450
 P 5800 3800
-F 0 "D?" H 5785 3870 24  0000 C CNN
+F 0 "D305" H 5785 3870 24  0000 C CNN
 F 1 "LED" H 5800 3700 50  0001 C CNN
 F 2 "~" H 5800 3800 60  0000 C CNN
@@
 $EndComp
 $Comp
-L LED D?
+L LED D304
 U 1 1 53A90456
 P 5650 3800
-F 0 "D?" H 5635 3870 24  0000 C CNN
+F 0 "D304" H 5635 3870 24  0000 C CNN
 F 1 "LED" H 5650 3700 50  0001 C CNN
 F 2 "~" H 5650 3800 60  0000 C CNN
@@
 $EndComp
 $Comp
-L LED D?
+L LED D303
 U 1 1 53A90466
 P 5500 3800
-F 0 "D?" H 5485 3870 24  0000 C CNN
+F 0 "D303" H 5485 3870 24  0000 C CNN
 F 1 "LED" H 5500 3700 50  0001 C CNN
 F 2 "~" H 5500 3800 60  0000 C CNN
@@
 $EndComp
 $Comp
-L LED D?
+L LED D302
 U 1 1 53A9046C
 P 5350 3800
-F 0 "D?" H 5335 3870 24  0000 C CNN
+F 0 "D302" H 5335 3870 24  0000 C CNN
 F 1 "LED" H 5350 3700 50  0001 C CNN
 F 2 "~" H 5350 3800 60  0000 C CNN
@@
 $EndComp
 $Comp
-L LED D?
+L LED D301
 U 1 1 53A90472
 P 5200 3800
-F 0 "D?" H 5185 3870 24  0000 C CNN
+F 0 "D301" H 5185 3870 24  0000 C CNN
 F 1 "LED" H 5200 3700 50  0001 C CNN
 F 2 "~" H 5200 3800 60  0000 C CNN
@@
 GND
 $Comp
-L R R?
+L R R307
 U 1 1 53A90918
 P 4850 2800
-F 0 "R?" V 4900 2600 40  0000 C CNN
+F 0 "R307" V 4900 2550 40  0000 C CNN
 F 1 "330" V 4857 2801 40  0000 C CNN
 F 2 "~" V 4780 2800 30  0000 C CNN
@@
 $EndComp
 $Comp
-L R R?
+L R R308
 U 1 1 53A90944
 P 4850 2900
-F 0 "R?" V 4900 2700 40  0000 C CNN
+F 0 "R308" V 4900 2650 40  0000 C CNN
 F 1 "330" V 4857 2901 40  0000 C CNN
 F 2 "~" V 4780 2900 30  0000 C CNN
@@
 $EndComp
 $Comp
-L R R?
+L R R309
 U 1 1 53A9094A
 P 4850 3000
-F 0 "R?" V 4900 2800 40  0000 C CNN
+F 0 "R309" V 4900 2750 40  0000 C CNN
 F 1 "330" V 4857 3001 40  0000 C CNN
 F 2 "~" V 4780 3000 30  0000 C CNN
@@
 $EndComp
 $Comp
-L R R?
+L R R310
 U 1 1 53A90950
 P 4850 3100
-F 0 "R?" V 4900 2900 40  0000 C CNN
+F 0 "R310" V 4900 2850 40  0000 C CNN
 F 1 "330" V 4857 3101 40  0000 C CNN
 F 2 "~" V 4780 3100 30  0000 C CNN
@@
 $EndComp
 $Comp
-L R R?
+L R R311
 U 1 1 53A90956
 P 4850 3200
-F 0 "R?" V 4900 3000 40  0000 C CNN
+F 0 "R311" V 4900 2950 40  0000 C CNN
 F 1 "330" V 4857 3201 40  0000 C CNN
 F 2 "~" V 4780 3200 30  0000 C CNN
@@
 $EndComp
 $Comp
-L R R?
+L R R312
 U 1 1 53A9095C
 P 4850 3300
-F 0 "R?" V 4900 3100 40  0000 C CNN
+F 0 "R312" V 4900 3050 40  0000 C CNN
 F 1 "330" V 4857 3301 40  0000 C CNN
 F 2 "~" V 4780 3300 30  0000 C CNN
@@
 $EndComp
 $Comp
-L R R?
+L R R313
 U 1 1 53A9096C
 P 4850 3400
-F 0 "R?" V 4900 3200 40  0000 C CNN
+F 0 "R313" V 4900 3150 40  0000 C CNN
 F 1 "330" V 4857 3401 40  0000 C CNN
 F 2 "~" V 4780 3400 30  0000 C CNN
@@
 $EndComp
 $Comp
-L R R?
+L R R314
 U 1 1 53A90972
 P 4850 3500
-F 0 "R?" V 4900 3300 40  0000 C CNN
+F 0 "R314" V 4900 3250 40  0000 C CNN
 F 1 "330" V 4857 3501 40  0000 C CNN
 F 2 "~" V 4780 3500 30  0000 C CNN
@@
 	6250 3500 6250 3600
 Wire Wire Line
-	4500 2400 4850 2400
-Wire Wire Line
-	4500 2300 4850 2300
-$Comp
-L CONN_2 P?
-U 1 1 53A9163A
-P 5250 2350
-F 0 "P?" V 5200 2350 40  0000 C CNN
-F 1 "UART2" V 5300 2350 40  0000 C CNN
-F 2 "" H 5250 2350 60  0000 C CNN
-F 3 "" H 5250 2350 60  0000 C CNN
-F 4 "1: RX 2: TX" H 5700 2250 60  0000 C CNN "Pinout"
-	1    5250 2350
+	4500 2400 5000 2400
+Wire Wire Line
+	4500 2300 5000 2300
+$Comp
+L CONN_4 P302
+U 1 1 53A91A1B
+P 5350 2350
+F 0 "P302" V 5300 2350 50  0000 C CNN
+F 1 "UART2" V 5400 2350 50  0000 C CNN
+F 2 "" H 5350 2350 60  0000 C CNN
+F 3 "" H 5350 2350 60  0000 C CNN
+	1    5350 2350
 	1    0    0    -1
 $EndComp
-Wire Wire Line
-	4850 2300 4900 2250
-Wire Wire Line
-	4850 2400 4900 2450
+Text Label 5000 2200 2    60   ~ 0
+VCC
+Text Label 5000 2500 2    60   ~ 0
+GND
 $EndSCHEMATC
