File: board/DTE - PIC18 USB.sch (KiCad schematic (older format))
At the start: 35 parts, among them J301 USB, P301 ICSP, P302 UART2, U301 PIC18F85J94, U302 AAT3221IGV-3.3-T1

Commit message: Major changes in DTE PIC18 USB sheet
Parts:
- removed P302: UART2, symbol CONN_4
- added C309: 8.2u, ~, symbol CSMALL
- added C310, C311: 22p, ~, symbol CSMALL
- added X301: CRYSTAL, ~, symbol CRYSTAL
Connections:
- wire segments 156 -> 137
Other:
- note added: "- First 4 serial ports use the 4 available hardware UARTs. Remaining serial ports need to be bitbanged\n\n- I2C is chosen to be bitbanged from RF6,7 \nbecause hardware I2C on RC5,6 and RD6,5 share pins with hardware UART. \n\n- It is preferable to have hardware support for UART since the I2C port will not be as heavily used as UART ports.\n\n- Crystal (and capactors) is optional.\nPIC18F85J94 has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"
- moved on the sheet: C307, D301, D302, D303, D304, D305, D306, D307, D308, J301, P301, R301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

Commit message: Fixed DRC errors in DTE PIC18 USB sheet, changed VCC names to include voltages
Parts:
- removed C309: 8.2u, ~, symbol CSMALL
- added C309: 8.2u, ~, symbol CP1
- X301: value CRYSTAL -> XTAL
Connections:
- net labels added: VCC_3V3, VCC_3v3
- wire segments 137 -> 139
Changed lines of the file:
@@
 Text HLabel 3950 4050 2    60   Input ~ 0
 DSR5
-Text HLabel 6750 1100 0    60   Output ~ 0
+Text HLabel 6500 1100 0    60   Output ~ 0
 5V
 Text HLabel 8350 3400 2    60   Input ~ 0
@@
 GND
 Text Label 8150 3200 2    60   ~ 0
-VCC
+VCC_3V3
 Text Label 2150 6250 1    60   ~ 0
-VCC
+VCC_3v3
 Text Label 5100 4450 0    60   ~ 0
-VCC
+VCC_3V3
 Text Label 2050 6250 1    60   ~ 0
 GND
@@
 PGC
 Text Label 1550 5850 2    60   ~ 0
-VCC
+VCC_3V3
 Text Label 8700 1450 0    60   ~ 0
-VCC
-Text Label 6700 2750 2    60   ~ 0
+VCC_3V3
+Text Label 6550 2750 2    60   ~ 0
 GND
 Text Label 4250 5000 0    60   ~ 0
-VCC
+VCC_3V3
 NoConn ~ 3800 5050
 NoConn ~ 3800 1650
@@
 NoConn ~ 3800 4150
 NoConn ~ 3800 4250
-Text Label 5700 3850 0    60   ~ 0
+Text Label 5800 3850 0    60   ~ 0
 GND
 $Comp
@@
 	6650 1450 7100 1450
 Wire Wire Line
-	6900 1100 6900 1850
-Connection ~ 6900 1450
+	7000 1450 7000 1850
+Connection ~ 7000 1450
 Wire Wire Line
 	6000 1600 6200 1600
@@
 Connection ~ 6150 2150
 Connection ~ 6150 2000
-Connection ~ 6700 1650
-Connection ~ 6700 2750
-Wire Wire Line
-	6900 1850 7100 1850
+Connection ~ 6550 1650
+Connection ~ 6550 2750
+Wire Wire Line
+	7000 1850 7100 1850
 Wire Wire Line
 	6000 2750 8700 2750
@@
 	1650 5850 1550 5850
 Wire Wire Line
-	6700 2750 6700 1650
+	6550 2750 6550 1650
 Wire Wire Line
 	4800 4800 4800 4650
@@
 NoConn ~ 3800 2250
 Wire Wire Line
-	6900 1100 6750 1100
-$Comp
-L CSMALL C309
-U 1 1 53AB15D3
-P 7000 1550
-F 0 "C309" H 7025 1600 30  0000 L CNN
-F 1 "8.2u" H 7025 1500 30  0000 L CNN
-F 2 "~" H 7000 1550 60  0000 C CNN
-F 3 "~" H 7000 1550 60  0000 C CNN
-	1    7000 1550
-	1    0    0    -1
-$EndComp
+	6800 1100 6500 1100
 Text Notes 5150 5900 0    60   ~ 0
 - First 4 serial ports use the 4 available hardware UARTs. Remaining serial ports need to be bitbanged\n\n- I2C is chosen to be bitbanged from RF6,7 \nbecause hardware I2C on RC5,6 and RD6,5 share pins with hardware UART. \n\n- It is preferable to have hardware support for UART since the I2C port will not be as heavily used as UART ports.\n\n- Crystal (and capactors) is optional.\nPIC18F85J94 has FRC internal clock, which is accurate enough to support USB 2.0 and UART.\n\n- LEDs on port H are optional and for debugging.
@@
 P 1400 2000
 F 0 "X301" H 1400 2150 60  0000 C CNN
-F 1 "CRYSTAL" H 1400 1850 60  0000 C CNN
+F 1 "XTAL" H 1400 1850 60  0000 C CNN
 F 2 "~" H 1400 2000 60  0000 C CNN
 F 3 "~" H 1400 2000 60  0000 C CNN
@@
 Text Label 800  2300 2    60   ~ 0
 GND
+$Comp
+L CP1 C309
+U 1 1 53AB30F6
+P 6800 2200
+F 0 "C309" H 6850 2300 50  0000 L CNN
+F 1 "8.2u" H 6850 2100 50  0000 L CNN
+F 2 "~" H 6800 2200 60  0000 C CNN
+F 3 "~" H 6800 2200 60  0000 C CNN
+	1    6800 2200
+	1    0    0    -1
+$EndComp
+Wire Wire Line
+	6800 1100 6800 2000
+Connection ~ 6800 1450
+Wire Wire Line
+	6800 2400 6800 2750
+Connection ~ 6800 2750
 $EndSCHEMATC

Commit message: Fixed power pin and port names to include voltages
Connections:
- net labels removed: VCC
Changed lines of the file:
@@
 GND
 Text HLabel 8350 3200 2    60   Output ~ 0
-VCC
+VCC_3V3
 Text HLabel 3950 1850 2    60   BiDi ~ 0
 SDA
@@
 Text Label 6550 2750 2    60   ~ 0
 GND
-Text Label 4250 5000 0    60   ~ 0
+Text Label 3900 4950 0    60   ~ 0
 VCC_3V3
 NoConn ~ 3800 5050
