File: board/Serial Expansion Motherboard.sch (KiCad schematic (older format))
At the start: 5 parts, among them U401 24AA014

Commit message: Fixed power pin and port names to include voltages
Connections:
- net labels added: +3.3V, VCC_3V3
- net labels removed: VCC
Changed lines of the file:
@@
 5V
 Text HLabel 4950 2000 0    60   Input ~ 0
-VCC
+VCC_3V3
 Text HLabel 1400 2150 0    60   Input ~ 0
 GND
@@
 F36 "DTR5" I L 6700 5550 60
 F37 "DSR5" O L 6700 5650 60
-F38 "VCC" I L 6700 2000 60
+F38 "VCC_5V_ISO" I L 6700 2000 47
 F39 "ID_SDA" B R 7650 2250 60
 F40 "ID_SCL" B R 7650 2150 60
-F41 "ID_3.3V" I R 7650 2000 60
+F41 "ID_3V3" I R 7650 2000 60
 F42 "ID_GND" I R 7650 5850 60
 F43 "RTS3" I L 6700 4150 60
@@
 F 3 "" H 1750 2550 60  0000 C CNN
 	1    1750 2550
-	1    0    0    -1
-$EndComp
-$Comp
-L VCC #PWR03
-U 1 1 53B14771
-P 5100 1400
-F 0 "#PWR03" H 5100 1500 30  0001 C CNN
-F 1 "VCC" H 5100 1500 30  0000 C CNN
-F 2 "" H 5100 1400 60  0000 C CNN
-F 3 "" H 5100 1400 60  0000 C CNN
-	1    5100 1400
 	1    0    0    -1
 $EndComp
@@
 	9950 2550 10100 2550
 Connection ~ 10100 2550
-$Comp
-L VCC #PWR09
-U 1 1 53B55B31
-P 8550 1400
-F 0 "#PWR09" H 8550 1500 30  0001 C CNN
-F 1 "VCC" H 8550 1500 30  0000 C CNN
-F 2 "" H 8550 1400 60  0000 C CNN
-F 3 "" H 8550 1400 60  0000 C CNN
-	1    8550 1400
-	1    0    0    -1
-$EndComp
 Text HLabel 8000 2450 3    60   BiDi ~ 0
 SDA
@@
 Connection ~ 8000 2150
 Connection ~ 8150 2250
-$Comp
-L VCC #PWR010
-U 1 1 53B5B188
-P 8000 1400
-F 0 "#PWR010" H 8000 1500 30  0001 C CNN
-F 1 "VCC" H 8000 1500 30  0000 C CNN
-F 2 "" H 8000 1400 60  0000 C CNN
-F 3 "" H 8000 1400 60  0000 C CNN
-	1    8000 1400
-	1    0    0    -1
-$EndComp
 $Comp
 L R R402
@@
 Wire Wire Line
 	8000 1500 8000 1400
-$Comp
-L VCC #PWR011
-U 1 1 53B5CDEE
-P 8150 1400
-F 0 "#PWR011" H 8150 1500 30  0001 C CNN
-F 1 "VCC" H 8150 1500 30  0000 C CNN
-F 2 "" H 8150 1400 60  0000 C CNN
-F 3 "" H 8150 1400 60  0000 C CNN
-	1    8150 1400
-	1    0    0    -1
-$EndComp
 Wire Wire Line
 	8150 1500 8150 1400
@@
 Wire Wire Line
 	7750 2000 7750 1400
-$Comp
-L VCC #PWR013
-U 1 1 53B6B29A
-P 7750 1400
-F 0 "#PWR013" H 7750 1500 30  0001 C CNN
-F 1 "VCC" H 7750 1500 30  0000 C CNN
-F 2 "" H 7750 1400 60  0000 C CNN
-F 3 "" H 7750 1400 60  0000 C CNN
-	1    7750 1400
-	1    0    0    -1
-$EndComp
 Wire Wire Line
 	7650 5850 7750 5850
@@
 	0    1    1    0
 $EndComp
+$Comp
+L +3.3V #PWR?
+U 1 1 53AC3183
+P 5100 1400
+F 0 "#PWR?" H 5100 1360 30  0001 C CNN
+F 1 "+3.3V" H 5100 1510 30  0000 C CNN
+F 2 "" H 5100 1400 60  0000 C CNN
+F 3 "" H 5100 1400 60  0000 C CNN
+	1    5100 1400
+	1    0    0    -1
+$EndComp
+$Comp
+L +3.3V #PWR?
+U 1 1 53AC95BE
+P 7750 1400
+F 0 "#PWR?" H 7750 1360 30  0001 C CNN
+F 1 "+3.3V" H 7750 1510 30  0000 C CNN
+F 2 "" H 7750 1400 60  0000 C CNN
+F 3 "" H 7750 1400 60  0000 C CNN
+	1    7750 1400
+	1    0    0    -1
+$EndComp
+$Comp
+L +3.3V #PWR?
+U 1 1 53AC9B85
+P 8000 1400
+F 0 "#PWR?" H 8000 1360 30  0001 C CNN
+F 1 "+3.3V" H 8000 1510 30  0000 C CNN
+F 2 "" H 8000 1400 60  0000 C CNN
+F 3 "" H 8000 1400 60  0000 C CNN
+	1    8000 1400
+	1    0    0    -1
+$EndComp
+$Comp
+L +3.3V #PWR?
+U 1 1 53AC9D02
+P 8150 1400
+F 0 "#PWR?" H 8150 1360 30  0001 C CNN
+F 1 "+3.3V" H 8150 1510 30  0000 C CNN
+F 2 "" H 8150 1400 60  0000 C CNN
+F 3 "" H 8150 1400 60  0000 C CNN
+	1    8150 1400
+	1    0    0    -1
+$EndComp
+$Comp
+L +3.3V #PWR?
+U 1 1 53ACA5A5
+P 8550 1400
+F 0 "#PWR?" H 8550 1360 30  0001 C CNN
+F 1 "+3.3V" H 8550 1510 30  0000 C CNN
+F 2 "" H 8550 1400 60  0000 C CNN
+F 3 "" H 8550 1400 60  0000 C CNN
+	1    8550 1400
+	1    0    0    -1
+$EndComp
 $EndSCHEMATC
