File: boards/Motherboard/DTE - PIC18 USB.sch (KiCad schematic (older format))
At the start: 38 parts, among them J301 USB, P301 ICSP, U301 PIC18F85J94, U302 AAT3221IGV-3.3-T1, X301 XTAL

Commit message: Changed I2C pins on PIC18F85J94 to use free Port G
Other:
- note added: "- First 4 serial ports use the 4 available hardware UARTs. Remaining serial ports need to be bitbanged\n\n- I2C is chosen to be bitbanged from RG0,1 \nbecause hardware I2C on RC5,6 and RD6,5 share pins with hardware UART. \n\n- It is preferable to have hardware support for UART since the I2C port will not be as heavily used as UART ports.\n\n- Crystal (and capactors) is optional.\nPIC18F85J94 has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"
- note removed: "- First 4 serial ports use the 4 available hardware UARTs. Remaining serial ports need to be bitbanged\n\n- I2C is chosen to be bitbanged from RF6,7 \nbecause hardware I2C on RC5,6 and RD6,5 share pins with hardware UART. \n\n- It is preferable to have hardware support for UART since the I2C port will not be as heavily used as UART ports.\n\n- Crystal (and capactors) is optional.\nPIC18F85J94 has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"
Changed lines of the file:
@@
 Text HLabel 8350 3200 2    60   Output ~ 0
 VCC_3V3
-Text HLabel 3950 1850 2    60   BiDi ~ 0
+Text HLabel 3950 2150 2    60   BiDi ~ 0
 SDA
-Text HLabel 3950 1750 2    60   BiDi ~ 0
+Text HLabel 3950 2050 2    60   BiDi ~ 0
 SCL
 $Comp
@@
 VCC_3V3
 NoConn ~ 3800 5050
-NoConn ~ 3800 1650
-NoConn ~ 3800 2050
 NoConn ~ 3800 2350
 NoConn ~ 3800 2450
@@
 	4100 1450 4250 1600
 Wire Wire Line
-	3950 1850 3800 1850
-Wire Wire Line
-	3950 1750 3800 1750
+	3950 2150 3800 2150
+Wire Wire Line
+	3950 2050 3800 2050
 Wire Wire Line
 	2250 6400 2250 5850
@@
 NoConn ~ 2350 4250
 NoConn ~ 2350 4350
-NoConn ~ 3800 2150
 NoConn ~ 3800 2250
 Wire Wire Line
 	6800 1100 6500 1100
 Text Notes 5150 5900 0    60   ~ 0
-- First 4 serial ports use the 4 available hardware UARTs. Remaining serial ports need to be bitbanged\n\n- I2C is chosen to be bitbanged from RF6,7 \nbecause hardware I2C on RC5,6 and RD6,5 share pins with hardware UART. \n\n- It is preferable to have hardware support for UART since the I2C port will not be as heavily used as UART ports.\n\n- Crystal (and capactors) is optional.\nPIC18F85J94 has FRC internal clock, which is accurate enough to support USB 2.0 and UART.\n\n- LEDs on port H are optional and for debugging.
+- First 4 serial ports use the 4 available hardware UARTs. Remaining serial ports need to be bitbanged\n\n- I2C is chosen to be bitbanged from RG0,1 \nbecause hardware I2C on RC5,6 and RD6,5 share pins with hardware UART. \n\n- It is preferable to have hardware support for UART since the I2C port will not be as heavily used as UART ports.\n\n- Crystal (and capactors) is optional.\nPIC18F85J94 has FRC internal clock, which is accurate enough to support USB 2.0 and UART.\n\n- LEDs on port H are optional and for debugging.
 $Comp
 L CRYSTAL X301
@@
 	6800 2400 6800 2750
 Connection ~ 6800 2750
+NoConn ~ 3800 1650
+NoConn ~ 3800 1750
+NoConn ~ 3800 1850
 $EndSCHEMATC

Commit message: Updated PIC18F USB pin mapping, connections to be made
Connections:
- net labels added: HEADER_1, LEDA0, LEDA1, LEDA2, LEDB0, LEDB1, LEDB2, LED_P, LED_Q, LED_R, SCK1_FPGA, SCK2_HEADER, SDI1_FPGA, SDO1_FPGA, SDO2_HEADER, SLOT3_LED1, SLOT3_LED2, SLOT4_LED1, SLOT4_LED2, SLOT5_LED1, SLOT5_LED2, SS1_FPGA, SS2_HEADER
- wire segments 139 -> 188
- no-connect marks 16 -> 1
Other:
- moved on the sheet: D301, D302, D303, D304, D305, D306, D307, D308, R307, R308, R309, R310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

Commit message: Updated templates of all dboards with commonalities of all dboards
Other:
- note added: "- First 4 serial ports use the 4 available hardware UARTs. Remaining serial ports need to be bitbanged\n\n- Crystal (and capactors) is optional.\nPIC18F85J94 has FRC internal clock, which is accurate enough to support USB 2.0 and UART."
- note removed: "- First 4 serial ports use the 4 available hardware UARTs. Remaining serial ports need to be bitbanged\n\n- I2C is chosen to be bitbanged from RG0,1 \nbecause hardware I2C on RC5,6 and RD6,5 share pins with hardware UART. \n\n- It is preferable to have hardware support for UART since the I2C port will not be as heavily used as UART ports.\n\n- Crystal (and capactors) is optional.\nPIC18F85J94 has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"
Changed lines of the file:
@@
 	0    -1   -1   0
 $EndComp
-Text Notes 5150 5900 0    60   ~ 0
-- First 4 serial ports use the 4 available hardware UARTs. Remaining serial ports need to be bitbanged\n\n- I2C is chosen to be bitbanged from RG0,1 \nbecause hardware I2C on RC5,6 and RD6,5 share pins with hardware UART. \n\n- It is preferable to have hardware support for UART since the I2C port will not be as heavily used as UART ports.\n\n- Crystal (and capactors) is optional.\nPIC18F85J94 has FRC internal clock, which is accurate enough to support USB 2.0 and UART.\n\n- LEDs on port H are optional and for debugging.
+Text Notes 5200 6350 0    60   ~ 0
+- First 4 serial ports use the 4 available hardware UARTs. Remaining serial ports need to be bitbanged\n\n- Crystal (and capactors) is optional.\nPIC18F85J94 has FRC internal clock, which is accurate enough to support USB 2.0 and UART.
 $Comp
 L CRYSTAL X301

Commit message: Updated PIC18 USB sheet, top sheet connections remaining
Parts:
- added D?: LED, ~, symbol LED
- added P?: SPI2, symbol CONN_6
- added R?: 330, ~, symbol R
Connections:
- net labels added: LED_A0, LED_A1, LED_A2, LED_B0, LED_B1, LED_B2, SDI2_HEADER
- net labels removed: HEADER_1
- wire segments 188 -> 171
Other:
- moved on the sheet: D301, D302, D303, D304, D305, D306, D307, D308, R307, R308, R309, R310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

Commit message: Change to 5 serial port; Connect Atlys and PIC18F SPI; Entire schematic updated
Parts:
- added D702, D703, D704, D705: LED, ~, symbol LED
- added R702, R703, R704, R705: 330, ~, symbol R
- gave numbers to parts that had none: 3
Connections:
- net labels added: SCK1, SDI1, SDO1, SS1
- net labels removed: CTS5, DSR5, DTR5, LEDA0, LEDA1, LEDA2, LEDB0, LEDB1, LEDB2, RTS5, RX5, SCK1_FPGA, SDI1_FPGA, SDO1_FPGA, SLOT5_LED1, SLOT5_LED2, SS1_FPGA, TX5
- wire segments 171 -> 162
- no-connect marks 1 -> 9
Other:
- moved on the sheet: D301, D302, D303, D304, D305, D306, D307, D308, D701, P706, R308, R309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

Commit message: Change all serial connections to use BUS
Parts:
- removed C301, C302, C304, C305, C306, C308: 0.1u, ~, symbol CSMALL
- removed C303: 10u, ~, symbol CSMALL
- removed C307: 4.7n, ~, symbol C
- removed C309: 8.2u, ~, symbol CP1
- removed C310, C311: 22p, ~, symbol CSMALL
- removed D301, D302, D303, D304, D305, D306, D307, D308, D701, D702, D703, D704, D705: LED, ~, symbol LED
- removed J301: USB, symbol USB
- removed P301: ICSP, symbol CONN_5
- removed P706: SPI2, symbol CONN_6
- removed R301: 10K, ~, symbol R
- removed R302, R303: 50, ~, symbol R
- removed R304: 1M, ~, symbol R
- removed R305: 0.47, ~, symbol R
- removed R306: 0.10, ~, symbol R
- removed R307, R308, R309, R310, R311, R312, R313, R314, R701, R702, R703, R704, R705: 330, ~, symbol R
- removed U301: PIC18F85J94, ~, symbol PIC18F85J94
- removed U302: AAT3221IGV-3.3-T1, ~, symbol AAT3221IGV-3.3-T1
- removed X301: XTAL, ~, symbol CRYSTAL
- added C613, C614: 22p, ~, symbol CSMALL
- added C615, C616, C618, C619, C620, C623: 0.1u, ~, symbol CSMALL
- added C617: 10u, ~, symbol CSMALL
- added C621: 4.7n, ~, symbol C
- added C622: 8.2u, ~, symbol CP1
- added D601, D602, D603, D604, D605, D606, D607, D608, D609, D610, D611, D612, D613: LED, ~, symbol LED
- added J601: USB, symbol USB
- added P601: ICSP, symbol CONN_5
- added P602: SPI2, symbol CONN_6
- added R619: 10K, ~, symbol R
- added R620, R621: 50, ~, symbol R
- added R640: 1M, ~, symbol R
- added R641: 0.47, ~, symbol R
- added R642, R661, R662, R663, R682, R683, R684, R685, R686, R687, R688, R689, R690: 330, ~, symbol R
- added R691: 0.10, ~, symbol R
- added U607: PIC18F85J94, ~, symbol PIC18F85J94
- added U608: AAT3221IGV-3.3-T1, ~, symbol AAT3221IGV-3.3-T1
- added X601: XTAL, ~, symbol CRYSTAL
Connections:
- net labels added: SERIAL0, SERIAL1, SERIAL10, SERIAL11, SERIAL12, SERIAL13, SERIAL14, SERIAL15, SERIAL16, SERIAL17, SERIAL18, SERIAL19, SERIAL2, SERIAL20, SERIAL21, SERIAL22, SERIAL23, SERIAL24, SERIAL25, SERIAL26, SERIAL27, SERIAL28, SERIAL29, SERIAL3, SERIAL4, SERIAL5, SERIAL6, SERIAL7, SERIAL8, SERIAL9, SERIAL[0..29]
- wire segments 162 -> 192
