File: boards/Motherboard/DTE - PIC18 USB.sch (KiCad schematic (older format))
At the start: 49 parts, among them J601 USB, P601 ICSP, P602 SPI2, U607 PIC18F85J94, U608 AAT3221IGV-3.3-T1, X601 XTAL

Commit message: Updated LED references in PIC18FUSB. Fixes #19
Parts:
- renumbered D601 to DS11, D602 to DS12, D603 to DS21, D604 to DS22, D605 to DS31, D606 to DS32, D607 to DS41, D608 to DS42, D609 to DS51, D610 to DS52
Connections:
- net labels added: SLOT1_LED1, SLOT1_LED2, SLOT2_LED1, SLOT2_LED2, SLOT5_LED1, SLOT5_LED2
- net labels removed: LED_A0, LED_A1, LED_A2, LED_B0, LED_B1, LED_B2
Changed lines of the file:
@@
 $EndComp
 $Comp
-L LED D608
+L LED DS42
 U 1 1 53BC15B1
 P 9100 4250
-F 0 "D608" H 9085 4320 24  0000 C CNN
+F 0 "DS42" H 9085 4320 24  0000 C CNN
 F 1 "LED" H 9100 4150 50  0001 C CNN
 F 2 "~" H 9100 4250 60  0000 C CNN
@@
 $EndComp
 $Comp
-L LED D607
+L LED DS41
 U 1 1 53BC15B2
 P 9100 4100
-F 0 "D607" H 9085 4170 24  0000 C CNN
+F 0 "DS41" H 9085 4170 24  0000 C CNN
 F 1 "LED" H 9100 4000 50  0001 C CNN
 F 2 "~" H 9100 4100 60  0000 C CNN
@@
 $EndComp
 $Comp
-L LED D606
+L LED DS32
 U 1 1 53BC15B3
 P 9100 3950
-F 0 "D606" H 9085 4020 24  0000 C CNN
+F 0 "DS32" H 9085 4020 24  0000 C CNN
 F 1 "LED" H 9100 3850 50  0001 C CNN
 F 2 "~" H 9100 3950 60  0000 C CNN
@@
 $EndComp
 $Comp
-L LED D605
+L LED DS31
 U 1 1 53BC15B4
 P 9100 3800
-F 0 "D605" H 9085 3870 24  0000 C CNN
+F 0 "DS31" H 9085 3870 24  0000 C CNN
 F 1 "LED" H 9100 3700 50  0001 C CNN
 F 2 "~" H 9100 3800 60  0000 C CNN
@@
 $EndComp
 $Comp
-L LED D604
+L LED DS22
 U 1 1 53BC15B5
 P 9100 3650
-F 0 "D604" H 9085 3720 24  0000 C CNN
+F 0 "DS22" H 9085 3720 24  0000 C CNN
 F 1 "LED" H 9100 3550 50  0001 C CNN
 F 2 "~" H 9100 3650 60  0000 C CNN
@@
 $EndComp
 $Comp
-L LED D603
+L LED DS21
 U 1 1 53BC15B6
 P 9100 3500
-F 0 "D603" H 9085 3570 24  0000 C CNN
+F 0 "DS21" H 9085 3570 24  0000 C CNN
 F 1 "LED" H 9100 3400 50  0001 C CNN
 F 2 "~" H 9100 3500 60  0000 C CNN
@@
 $EndComp
 $Comp
-L LED D602
+L LED DS12
 U 1 1 53BC15B7
 P 9100 3350
-F 0 "D602" H 9085 3420 24  0000 C CNN
+F 0 "DS12" H 9085 3420 24  0000 C CNN
 F 1 "LED" H 9100 3250 50  0001 C CNN
 F 2 "~" H 9100 3350 60  0000 C CNN
@@
 $EndComp
 $Comp
-L LED D601
+L LED DS11
 U 1 1 53BC15B8
 P 9100 3200
-F 0 "D601" H 9085 3270 24  0000 C CNN
+F 0 "DS11" H 9085 3270 24  0000 C CNN
 F 1 "LED" H 9100 3100 50  0001 C CNN
 F 2 "~" H 9100 3200 60  0000 C CNN
@@
 $EndComp
 Text Label 3400 3100 2    60   ~ 0
-LED_A0
+SLOT1_LED1
 Text Label 3400 3200 2    60   ~ 0
-LED_B0
+SLOT1_LED2
 Text Label 3400 3300 2    60   ~ 0
-LED_A1
+SLOT2_LED1
 Text Label 3400 3600 2    60   ~ 0
-LED_B1
+SLOT2_LED2
 Text Label 3400 3700 2    60   ~ 0
-LED_A2
+SLOT3_LED1
 Text Label 3400 3800 2    60   ~ 0
-LED_B2
+SLOT3_LED2
 Text Label 3400 4100 2    60   ~ 0
 SDI2_HEADER
 Text Label 5650 1700 0    60   ~ 0
-SLOT3_LED1
+SLOT4_LED1
 Text Label 5650 1800 0    60   ~ 0
-SLOT3_LED2
+SLOT4_LED2
 $Comp
 L PIC18F85J94 U607
@@
 SDO2_HEADER
 Text Label 6100 3200 0    60   ~ 0
-SLOT4_LED1
+SLOT5_LED1
 Text Label 6100 3300 0    60   ~ 0
-SLOT4_LED2
+SLOT5_LED2
 Text Label 3400 4000 2    60   ~ 0
 LED_P
@@
 LED_R
 $Comp
-L LED D609
+L LED DS51
 U 1 1 53BC15C6
 P 9100 4400
-F 0 "D609" H 9085 4470 24  0000 C CNN
+F 0 "DS51" H 9085 4470 24  0000 C CNN
 F 1 "LED" H 9100 4300 50  0001 C CNN
 F 2 "~" H 9100 4400 60  0000 C CNN
@@
 $EndComp
 Text Label 8100 3200 2    60   ~ 0
-LED_A0
+SLOT1_LED1
 Text Label 8100 3350 2    60   ~ 0
-LED_A1
+SLOT1_LED2
 Text Label 8100 3500 2    60   ~ 0
-LED_A2
+SLOT2_LED1
 Text Label 8100 3650 2    60   ~ 0
-LED_B0
+SLOT2_LED2
 Text Label 8100 3800 2    60   ~ 0
-LED_B1
+SLOT3_LED1
 Text Label 8100 3950 2    60   ~ 0
-LED_B2
-Text Label 8100 4100 2    60   ~ 0
+SLOT3_LED2
+Text Label 8100 4700 2    60   ~ 0
 LED_P
-Text Label 8100 4250 2    60   ~ 0
+Text Label 8100 4850 2    60   ~ 0
 LED_Q
-Text Label 8100 4400 2    60   ~ 0
+Text Label 8100 5000 2    60   ~ 0
 LED_R
 $Comp
@@
 $EndComp
 $Comp
-L LED D610
+L LED DS52
 U 1 1 53BC15CB
 P 9100 4550
-F 0 "D610" H 9085 4620 24  0000 C CNN
+F 0 "DS52" H 9085 4620 24  0000 C CNN
 F 1 "LED" H 9100 4450 50  0001 C CNN
 F 2 "~" H 9100 4550 60  0000 C CNN
@@
 	0    -1   -1   0
 $EndComp
+Text Label 8100 4100 2    60   ~ 0
+SLOT4_LED1
+Text Label 8100 4250 2    60   ~ 0
+SLOT4_LED2
+Text Label 8100 4400 2    60   ~ 0
+SLOT5_LED1
 Text Label 8100 4550 2    60   ~ 0
-SLOT3_LED1
-Text Label 8100 4700 2    60   ~ 0
-SLOT3_LED2
-Text Label 8100 4850 2    60   ~ 0
-SLOT4_LED1
-Text Label 8100 5000 2    60   ~ 0
-SLOT4_LED2
+SLOT5_LED2
 Wire Wire Line
 	5450 1300 5650 1300
@@
 	8450 1050 8150 1050
 Wire Wire Line
-	8100 4250 8250 4250
-Wire Wire Line
-	8250 4100 8100 4100
+	8100 4850 8250 4850
+Wire Wire Line
+	8250 4700 8100 4700
 Wire Wire Line
 	8100 3950 8250 3950
@@
 	4000 4000 3400 4000
 Wire Wire Line
-	8250 4400 8100 4400
+	8250 5000 8100 5000
 Wire Wire Line
 	5450 2000 6250 2000
@@
 	8750 4400 8900 4400
 Wire Wire Line
-	8100 4850 8250 4850
-Wire Wire Line
-	8250 4700 8100 4700
-Wire Wire Line
-	8100 4550 8250 4550
-Wire Wire Line
-	8250 5000 8100 5000
+	8100 4400 8250 4400
+Wire Wire Line
+	8250 4250 8100 4250
+Wire Wire Line
+	8100 4100 8250 4100
+Wire Wire Line
+	8250 4550 8100 4550
 Wire Wire Line
 	8900 4550 8750 4550

Commit message: Changed LED resistor references in PIC18F USB sheet
Parts:
- renumbered R642 to RS11, R661 to RS12, R662 to RS21, R663 to RS22, R682 to RS31, R683 to RS32, R684 to RS41, R685 to RS42, R686 to RS51, R687 to RS52
Changed lines of the file:
@@
 GND
 $Comp
-L R R642
+L R RS11
 U 1 1 53BC15B9
 P 8500 3200
-F 0 "R642" V 8550 2950 40  0000 C CNN
+F 0 "RS11" V 8550 2950 40  0000 C CNN
 F 1 "330" V 8507 3201 40  0000 C CNN
 F 2 "~" V 8430 3200 30  0000 C CNN
@@
 $EndComp
 $Comp
-L R R661
+L R RS12
 U 1 1 53BC15BA
 P 8500 3350
-F 0 "R661" V 8550 3100 40  0000 C CNN
+F 0 "RS12" V 8550 3100 40  0000 C CNN
 F 1 "330" V 8507 3351 40  0000 C CNN
 F 2 "~" V 8430 3350 30  0000 C CNN
@@
 $EndComp
 $Comp
-L R R662
+L R RS21
 U 1 1 53BC15BB
 P 8500 3500
-F 0 "R662" V 8550 3250 40  0000 C CNN
+F 0 "RS21" V 8550 3250 40  0000 C CNN
 F 1 "330" V 8507 3501 40  0000 C CNN
 F 2 "~" V 8430 3500 30  0000 C CNN
@@
 $EndComp
 $Comp
-L R R663
+L R RS22
 U 1 1 53BC15BC
 P 8500 3650
-F 0 "R663" V 8550 3400 40  0000 C CNN
+F 0 "RS22" V 8550 3400 40  0000 C CNN
 F 1 "330" V 8507 3651 40  0000 C CNN
 F 2 "~" V 8430 3650 30  0000 C CNN
@@
 $EndComp
 $Comp
-L R R682
+L R RS31
 U 1 1 53BC15BD
 P 8500 3800
-F 0 "R682" V 8550 3550 40  0000 C CNN
+F 0 "RS31" V 8550 3550 40  0000 C CNN
 F 1 "330" V 8507 3801 40  0000 C CNN
 F 2 "~" V 8430 3800 30  0000 C CNN
@@
 $EndComp
 $Comp
-L R R683
+L R RS32
 U 1 1 53BC15BE
 P 8500 3950
-F 0 "R683" V 8550 3700 40  0000 C CNN
+F 0 "RS32" V 8550 3700 40  0000 C CNN
 F 1 "330" V 8507 3951 40  0000 C CNN
 F 2 "~" V 8430 3950 30  0000 C CNN
@@
 $EndComp
 $Comp
-L R R684
+L R RS41
 U 1 1 53BC15BF
 P 8500 4100
-F 0 "R684" V 8550 3850 40  0000 C CNN
+F 0 "RS41" V 8550 3850 40  0000 C CNN
 F 1 "330" V 8507 4101 40  0000 C CNN
 F 2 "~" V 8430 4100 30  0000 C CNN
@@
 $EndComp
 $Comp
-L R R685
+L R RS42
 U 1 1 53BC15C0
 P 8500 4250
-F 0 "R685" V 8550 4000 40  0000 C CNN
+F 0 "RS42" V 8550 4000 40  0000 C CNN
 F 1 "330" V 8507 4251 40  0000 C CNN
 F 2 "~" V 8430 4250 30  0000 C CNN
@@
 $EndComp
 $Comp
-L R R686
+L R RS51
 U 1 1 53BC15C7
 P 8500 4400
-F 0 "R686" V 8550 4150 40  0000 C CNN
+F 0 "RS51" V 8550 4150 40  0000 C CNN
 F 1 "330" V 8507 4401 40  0000 C CNN
 F 2 "~" V 8430 4400 30  0000 C CNN
@@
 $EndComp
 $Comp
-L R R687
+L R RS52
 U 1 1 53BC15CC
 P 8500 4550
-F 0 "R687" V 8550 4300 40  0000 C CNN
+F 0 "RS52" V 8550 4300 40  0000 C CNN
 F 1 "330" V 8507 4551 40  0000 C CNN
 F 2 "~" V 8430 4550 30  0000 C CNN

Commit message: Changed C622 to use std value MLCC
Parts:
- removed C622: 8.2u, ~, symbol CP1
- added C622: 4.7u, ~, symbol C
Changed lines of the file:
@@
 Text Label 2750 2100 2    60   ~ 0
 GND
-$Comp
-L CP1 C622
-U 1 1 53BC15C4
-P 8450 2150
-F 0 "C622" H 8500 2250 50  0000 L CNN
-F 1 "8.2u" H 8500 2050 50  0000 L CNN
-F 2 "~" H 8450 2150 60  0000 C CNN
-F 3 "~" H 8450 2150 60  0000 C CNN
-	1    8450 2150
-	1    0    0    -1
-$EndComp
 Text Label 3400 3100 2    60   ~ 0
 SLOT1_LED1
@@
 Text Label 1700 6750 0    60   ~ 0
 SLOT55
+$Comp
+L C C622
+U 1 1 53B40107
+P 8450 2150
+F 0 "C622" H 8450 2250 40  0000 L CNN
+F 1 "4.7u" H 8456 2065 40  0000 L CNN
+F 2 "~" H 8488 2000 30  0000 C CNN
+F 3 "~" H 8450 2150 60  0000 C CNN
+	1    8450 2150
+	1    0    0    -1
+$EndComp
 $EndSCHEMATC

Commit message: Changed LED resistor values to 1.5k in PIC18 USB schematic
Parts:
- R688, R689, R690, RS11, RS12, RS21, RS22, RS31, RS32, RS41, RS42, RS51, RS52: value 330 -> 1.5k
Changed lines of the file:
@@
 Sheet 7 7
 Title ""
-Date "2 jul 2014"
+Date "3 jul 2014"
 Rev ""
 Comp "TimVideos"
@@
 P 8500 3200
 F 0 "RS11" V 8550 2950 40  0000 C CNN
-F 1 "330" V 8507 3201 40  0000 C CNN
+F 1 "1.5k" V 8507 3201 40  0000 C CNN
 F 2 "~" V 8430 3200 30  0000 C CNN
 F 3 "~" H 8500 3200 30  0000 C CNN
@@
 P 8500 3350
 F 0 "RS12" V 8550 3100 40  0000 C CNN
-F 1 "330" V 8507 3351 40  0000 C CNN
+F 1 "1.5k" V 8507 3351 40  0000 C CNN
 F 2 "~" V 8430 3350 30  0000 C CNN
 F 3 "~" H 8500 3350 30  0000 C CNN
@@
 P 8500 3500
 F 0 "RS21" V 8550 3250 40  0000 C CNN
-F 1 "330" V 8507 3501 40  0000 C CNN
+F 1 "1.5k" V 8507 3501 40  0000 C CNN
 F 2 "~" V 8430 3500 30  0000 C CNN
 F 3 "~" H 8500 3500 30  0000 C CNN
@@
 P 8500 3650
 F 0 "RS22" V 8550 3400 40  0000 C CNN
-F 1 "330" V 8507 3651 40  0000 C CNN
+F 1 "1.5k" V 8507 3651 40  0000 C CNN
 F 2 "~" V 8430 3650 30  0000 C CNN
 F 3 "~" H 8500 3650 30  0000 C CNN
@@
 P 8500 3800
 F 0 "RS31" V 8550 3550 40  0000 C CNN
-F 1 "330" V 8507 3801 40  0000 C CNN
+F 1 "1.5k" V 8507 3801 40  0000 C CNN
 F 2 "~" V 8430 3800 30  0000 C CNN
 F 3 "~" H 8500 3800 30  0000 C CNN
@@
 P 8500 3950
 F 0 "RS32" V 8550 3700 40  0000 C CNN
-F 1 "330" V 8507 3951 40  0000 C CNN
+F 1 "1.5k" V 8507 3951 40  0000 C CNN
 F 2 "~" V 8430 3950 30  0000 C CNN
 F 3 "~" H 8500 3950 30  0000 C CNN
@@
 P 8500 4100
 F 0 "RS41" V 8550 3850 40  0000 C CNN
-F 1 "330" V 8507 4101 40  0000 C CNN
+F 1 "1.5k" V 8507 4101 40  0000 C CNN
 F 2 "~" V 8430 4100 30  0000 C CNN
 F 3 "~" H 8500 4100 30  0000 C CNN
@@
 P 8500 4250
 F 0 "RS42" V 8550 4000 40  0000 C CNN
-F 1 "330" V 8507 4251 40  0000 C CNN
+F 1 "1.5k" V 8507 4251 40  0000 C CNN
 F 2 "~" V 8430 4250 30  0000 C CNN
 F 3 "~" H 8500 4250 30  0000 C CNN
@@
 P 8500 4400
 F 0 "RS51" V 8550 4150 40  0000 C CNN
-F 1 "330" V 8507 4401 40  0000 C CNN
+F 1 "1.5k" V 8507 4401 40  0000 C CNN
 F 2 "~" V 8430 4400 30  0000 C CNN
 F 3 "~" H 8500 4400 30  0000 C CNN
@@
 P 8500 4550
 F 0 "RS52" V 8550 4300 40  0000 C CNN
-F 1 "330" V 8507 4551 40  0000 C CNN
+F 1 "1.5k" V 8507 4551 40  0000 C CNN
 F 2 "~" V 8430 4550 30  0000 C CNN
 F 3 "~" H 8500 4550 30  0000 C CNN
@@
 P 8500 4700
 F 0 "R688" V 8550 4450 40  0000 C CNN
-F 1 "330" V 8507 4701 40  0000 C CNN
+F 1 "1.5k" V 8507 4701 40  0000 C CNN
 F 2 "~" V 8430 4700 30  0000 C CNN
 F 3 "~" H 8500 4700 30  0000 C CNN
@@
 P 8500 4850
 F 0 "R689" V 8550 4600 40  0000 C CNN
-F 1 "330" V 8507 4851 40  0000 C CNN
+F 1 "1.5k" V 8507 4851 40  0000 C CNN
 F 2 "~" V 8430 4850 30  0000 C CNN
 F 3 "~" H 8500 4850 30  0000 C CNN
@@
 P 8500 5000
 F 0 "R690" V 8550 4750 40  0000 C CNN
-F 1 "330" V 8507 5001 40  0000 C CNN
+F 1 "1.5k" V 8507 5001 40  0000 C CNN
 F 2 "~" V 8430 5000 30  0000 C CNN
 F 3 "~" H 8500 5000 30  0000 C CNN

Commit message: Changed LED resistor to 680R in PIC18 USB
Parts:
- R688, R689, R690, RS11, RS12, RS21, RS22, RS31, RS32, RS41, RS42, RS51, RS52: value 1.5k -> 680
Changed lines of the file:
@@
 Sheet 7 7
 Title ""
-Date "3 jul 2014"
+Date "4 jul 2014"
 Rev ""
 Comp "TimVideos"
@@
 P 8500 3200
 F 0 "RS11" V 8550 2950 40  0000 C CNN
-F 1 "1.5k" V 8507 3201 40  0000 C CNN
+F 1 "680" V 8507 3201 40  0000 C CNN
 F 2 "~" V 8430 3200 30  0000 C CNN
 F 3 "~" H 8500 3200 30  0000 C CNN
@@
 P 8500 3350
 F 0 "RS12" V 8550 3100 40  0000 C CNN
-F 1 "1.5k" V 8507 3351 40  0000 C CNN
+F 1 "680" V 8507 3351 40  0000 C CNN
 F 2 "~" V 8430 3350 30  0000 C CNN
 F 3 "~" H 8500 3350 30  0000 C CNN
@@
 P 8500 3500
 F 0 "RS21" V 8550 3250 40  0000 C CNN
-F 1 "1.5k" V 8507 3501 40  0000 C CNN
+F 1 "680" V 8507 3501 40  0000 C CNN
 F 2 "~" V 8430 3500 30  0000 C CNN
 F 3 "~" H 8500 3500 30  0000 C CNN
@@
 P 8500 3650
 F 0 "RS22" V 8550 3400 40  0000 C CNN
-F 1 "1.5k" V 8507 3651 40  0000 C CNN
+F 1 "680" V 8507 3651 40  0000 C CNN
 F 2 "~" V 8430 3650 30  0000 C CNN
 F 3 "~" H 8500 3650 30  0000 C CNN
@@
 P 8500 3800
 F 0 "RS31" V 8550 3550 40  0000 C CNN
-F 1 "1.5k" V 8507 3801 40  0000 C CNN
+F 1 "680" V 8507 3801 40  0000 C CNN
 F 2 "~" V 8430 3800 30  0000 C CNN
 F 3 "~" H 8500 3800 30  0000 C CNN
@@
 P 8500 3950
 F 0 "RS32" V 8550 3700 40  0000 C CNN
-F 1 "1.5k" V 8507 3951 40  0000 C CNN
+F 1 "680" V 8507 3951 40  0000 C CNN
 F 2 "~" V 8430 3950 30  0000 C CNN
 F 3 "~" H 8500 3950 30  0000 C CNN
@@
 P 8500 4100
 F 0 "RS41" V 8550 3850 40  0000 C CNN
-F 1 "1.5k" V 8507 4101 40  0000 C CNN
+F 1 "680" V 8507 4101 40  0000 C CNN
 F 2 "~" V 8430 4100 30  0000 C CNN
 F 3 "~" H 8500 4100 30  0000 C CNN
@@
 P 8500 4250
 F 0 "RS42" V 8550 4000 40  0000 C CNN
-F 1 "1.5k" V 8507 4251 40  0000 C CNN
+F 1 "680" V 8507 4251 40  0000 C CNN
 F 2 "~" V 8430 4250 30  0000 C CNN
 F 3 "~" H 8500 4250 30  0000 C CNN
@@
 P 8500 4400
 F 0 "RS51" V 8550 4150 40  0000 C CNN
-F 1 "1.5k" V 8507 4401 40  0000 C CNN
+F 1 "680" V 8507 4401 40  0000 C CNN
 F 2 "~" V 8430 4400 30  0000 C CNN
 F 3 "~" H 8500 4400 30  0000 C CNN
@@
 P 8500 4550
 F 0 "RS52" V 8550 4300 40  0000 C CNN
-F 1 "1.5k" V 8507 4551 40  0000 C CNN
+F 1 "680" V 8507 4551 40  0000 C CNN
 F 2 "~" V 8430 4550 30  0000 C CNN
 F 3 "~" H 8500 4550 30  0000 C CNN
@@
 P 8500 4700
 F 0 "R688" V 8550 4450 40  0000 C CNN
-F 1 "1.5k" V 8507 4701 40  0000 C CNN
+F 1 "680" V 8507 4701 40  0000 C CNN
 F 2 "~" V 8430 4700 30  0000 C CNN
 F 3 "~" H 8500 4700 30  0000 C CNN
@@
 P 8500 4850
 F 0 "R689" V 8550 4600 40  0000 C CNN
-F 1 "1.5k" V 8507 4851 40  0000 C CNN
+F 1 "680" V 8507 4851 40  0000 C CNN
 F 2 "~" V 8430 4850 30  0000 C CNN
 F 3 "~" H 8500 4850 30  0000 C CNN
@@
 P 8500 5000
 F 0 "R690" V 8550 4750 40  0000 C CNN
-F 1 "1.5k" V 8507 5001 40  0000 C CNN
+F 1 "680" V 8507 5001 40  0000 C CNN
 F 2 "~" V 8430 5000 30  0000 C CNN
 F 3 "~" H 8500 5000 30  0000 C CNN
