File: boards/Motherboard/Data isolation.sch (KiCad schematic (older format))
At the start: 102 parts, among them U601 SI8660, U602 SI8660, U603 SI8660, U604 SI8660, U605 SI8660, U606 SI8660

Commit message: Change to 5 serial port; Connect Atlys and PIC18F SPI; Entire schematic updated
Parts:
- removed R619, R620, R621, R640, R641, R642, R661, R662, R663, R682, R683, R684: 100, ~, symbol R
Connections:
- net labels removed: IN15_A, IN15_B, IN16_A, IN16_B, IN17_A, IN17_B, OUT15_A, OUT15_B, OUT16_A, OUT16_B, OUT17_A, OUT17_B
- wire segments 216 -> 192
- no-connect marks 0 -> 12
