File: boards/Motherboard/Data isolation.sch (KiCad schematic (older format))
At the start: 90 parts, among them U601 SI8660, U602 SI8660, U603 SI8660, U604 SI8660, U605 SI8660, U606 SI8660

Commit message: Changed U606 value to include Si8630
Parts:
- U605: renamed from U603; value SI8660 -> SI8630/SI8660
- U606: value SI8660 -> SI8630/SI8660
- renumbered U604 to U602, U602 to U603, U605 to U604
Other:
- moved on the sheet: R616, R617, R618, R637, R638, R639, R658, R659, R660, R679, R680, R681

Commit message: Flipped U602, U604, U606 in data isolation sheet to make it less confusing, fixed typo in note written below
Other:
- note added: "Postfix A refers to DTE side and postfix B refers to daughterboard side.\ne.g. IN12_A is an input for DTE side and OUT12_B is the corresponding output to daughterboard side.\n"
- note removed: "Postfix A refers to DTE side and postfix B refers to daughterboard side.\ne.g. IN12_A in an input from DTE side and OUT12_B is the output connected to daughterboard side.\n"
- moved on the sheet: R643, R644, R645, R646, R647, R648, R649, R650, R651, R652, R653, R654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
