File: boards/GPIO-8 daughterboard/GPIO-8 standalone.sch (KiCad schematic (older format))
At the start: 13 parts, among them J201 DB9, J202 DB9, U201 ISL83387E, U202 24AA014

Commit message: GPIO-8 daughterboard done; create reusable PIC16F GPIO sheet
Parts:
- removed J202: DB9, symbol DB9
- added P201: GPIO_HEADER, symbol CONN_10
Connections:
- net labels removed: C_CTS, C_DSR, C_DTR, C_RTS, C_RX, C_TX
- wire segments 90 -> 92
- no-connect marks 4 -> 2
Changed lines of the file:
@@
 LIBS:csmall
 LIBS:ISL83387E
+LIBS:pic16f1704
 LIBS:GPIO-8 daughterboard-cache
 EELAYER 27 0
@@
 $Descr A4 11693 8268
 encoding utf-8
-Sheet 2 2
+Sheet 2 3
 Title ""
 Date "26 jun 2014"
@@
 Text Label 2550 3650 2    60   ~ 0
 A_DSR
-Text Label 10100 3250 2    60   ~ 0
-C_DTR
-Text Label 10100 3350 2    60   ~ 0
-C_CTS
-Text Label 10100 3450 2    60   ~ 0
-C_TX
-Text Label 10100 3550 2    60   ~ 0
-C_RTS
-Text Label 10100 3650 2    60   ~ 0
-C_RX
-Text Label 10100 3750 2    60   ~ 0
-C_DSR
 Text Label 5350 3250 0    60   ~ 0
 B_RX
@@
 Text Label 5350 3750 0    60   ~ 0
 B_DTR
-Text Label 6300 3350 2    60   ~ 0
+Text Label 6950 3350 2    60   ~ 0
 B_RX
-Text Label 6300 3250 2    60   ~ 0
+Text Label 6950 3250 2    60   ~ 0
 B_TX
-Text Label 6300 3450 2    60   ~ 0
-B_RTS
-Text Label 6300 3550 2    60   ~ 0
-B_CTS
-Text Label 6300 3650 2    60   ~ 0
-B_DTR
-Text Label 6300 3750 2    60   ~ 0
-B_DSR
 Text Label 6000 2700 3    60   ~ 0
 B_RX
@@
 Text Label 5600 2700 3    60   ~ 0
 B_DSR
-NoConn ~ 10250 3850
-NoConn ~ 10250 3150
-$Comp
-L DB9 J202
-U 1 1 53ABD89D
-P 10700 3450
-F 0 "J202" H 10700 4000 70  0000 C CNN
-F 1 "DB9" H 10700 2900 70  0000 C CNN
-F 2 "" H 10700 3450 60  0000 C CNN
-F 3 "" H 10700 3450 60  0000 C CNN
-	1    10700 3450
-	1    0    0    -1
-$EndComp
 Wire Wire Line
 	4800 6450 4700 6450
@@
 	5500 6050 5500 6150
 Wire Wire Line
-	6950 3250 6300 3250
-Wire Wire Line
-	6950 3350 6300 3350
-Wire Wire Line
-	6950 3450 6300 3450
-Wire Wire Line
-	6950 3550 6300 3550
-Wire Wire Line
-	6950 3650 6300 3650
-Wire Wire Line
-	6950 3750 6300 3750
+	7100 3250 6950 3250
+Wire Wire Line
+	7100 3350 6950 3350
 Wire Wire Line
 	2750 2650 2750 2600
@@
 Wire Wire Line
 	5600 2350 5600 2700
-Wire Wire Line
-	10250 3650 10100 3650
-Wire Wire Line
-	10250 3250 10100 3250
-Wire Wire Line
-	10250 3350 10100 3350
-Wire Wire Line
-	10250 3750 10100 3750
-Wire Wire Line
-	10250 3450 10100 3450
-Wire Wire Line
-	10250 3550 10100 3550
-$Comp
-L PWR_FLAG #FLG201
+$Comp
+L PWR_FLAG #FLG01
 U 1 1 53ABE834
 P 2950 2350
-F 0 "#FLG201" H 2950 2445 30  0001 C CNN
+F 0 "#FLG01" H 2950 2445 30  0001 C CNN
 F 1 "PWR_FLAG" H 2950 2530 30  0001 C CNN
 F 2 "" H 2950 2350 60  0000 C CNN
@@
 $EndComp
 $Comp
-L PWR_FLAG #FLG202
+L PWR_FLAG #FLG02
 U 1 1 53ABE907
 P 5500 6050
-F 0 "#FLG202" H 5500 6145 30  0001 C CNN
+F 0 "#FLG02" H 5500 6145 30  0001 C CNN
 F 1 "PWR_FLAG" H 5500 6230 30  0001 C CNN
 F 2 "" H 5500 6050 60  0000 C CNN
@@
 $EndComp
 $Comp
-L PWR_FLAG #FLG203
+L PWR_FLAG #FLG03
 U 1 1 53ABE910
 P 7050 6050
-F 0 "#FLG203" H 7050 6145 30  0001 C CNN
+F 0 "#FLG03" H 7050 6145 30  0001 C CNN
 F 1 "PWR_FLAG" H 7050 6230 30  0001 C CNN
 F 2 "" H 7050 6050 60  0000 C CNN
@@
 $EndComp
 $Comp
-L PWR_FLAG #FLG204
+L PWR_FLAG #FLG04
 U 1 1 53ABE916
 P 7050 6550
-F 0 "#FLG204" H 7050 6645 30  0001 C CNN
+F 0 "#FLG04" H 7050 6645 30  0001 C CNN
 F 1 "PWR_FLAG" H 7050 6730 30  0001 C CNN
 F 2 "" H 7050 6550 60  0000 C CNN
@@
 Wire Wire Line
 	1700 3150 1700 3000
-Wire Wire Line
-	10250 3050 10100 3050
-Text HLabel 10100 2900 1    60   Input ~ 0
-GND_ISO
-Wire Wire Line
-	10100 3050 10100 2900
 $Comp
 L R R203
@@
 Wire Wire Line
 	4800 6050 4700 6050
+Wire Wire Line
+	7100 3100 6950 3100
+Text Label 6950 3100 2    60   ~ 0
+VCC_5V_ISO
+Wire Wire Line
+	7100 3500 6950 3500
+Text Label 6950 3500 2    60   ~ 0
+GND_ISO
+$Comp
+L CONN_10 P201
+U 1 1 53ACAF9C
+P 8650 3550
+F 0 "P201" V 8600 3550 60  0000 C CNN
+F 1 "GPIO_HEADER" V 8700 3550 60  0000 C CNN
+F 2 "" H 8650 3550 60  0000 C CNN
+F 3 "" H 8650 3550 60  0000 C CNN
+	1    8650 3550
+	1    0    0    -1
+$EndComp
+Wire Wire Line
+	8300 3100 7950 3100
+Wire Wire Line
+	8300 3200 7950 3200
+Wire Wire Line
+	8300 3300 7950 3300
+Wire Wire Line
+	8300 3400 7950 3400
+Wire Wire Line
+	8300 3500 7950 3500
+Wire Wire Line
+	8300 3600 7950 3600
+Wire Wire Line
+	8300 3700 7950 3700
+Wire Wire Line
+	8300 3800 7950 3800
+Wire Wire Line
+	8300 4000 8200 4000
+Text Label 8200 4300 2    60   ~ 0
+VCC_5V_ISO
+Wire Wire Line
+	8200 4000 8200 4300
+Wire Wire Line
+	8300 3900 8050 3900
+Wire Wire Line
+	8050 3900 8050 4150
+Text Label 8050 4150 2    60   ~ 0
+GND_ISO
+$Sheet
+S 7100 3000 850  900
+U 53AC80BA
+F0 "PIC-GPIO8.sch" 50
+F1 "PIC-GPIO8.sch" 50
+F2 "VCC" I L 7100 3100 60
+F3 "GND" I L 7100 3500 60
+F4 "GPIO0" B R 7950 3100 60
+F5 "GPIO1" B R 7950 3200 60
+F6 "GPIO2" B R 7950 3300 60
+F7 "GPIO5" B R 7950 3600 60
+F8 "GPIO6" B R 7950 3700 60
+F9 "GPIO7" B R 7950 3800 60
+F10 "GPIO4" B R 7950 3500 60
+F11 "GPIO3" B R 7950 3400 60
+F12 "RX" I L 7100 3350 60
+F13 "TX" O L 7100 3250 60
+$EndSheet
 $EndSCHEMATC

Commit message: Updated GPIO8 dboard to use RS232 adapter block; Changed power hierarchy pin in RS232_adapter_block and PIC-GPIO8 sheets as passive type
Parts:
- removed C201, C202, C203, C204, C205, C206: 0.1u, ~, symbol CSMALL
- removed D201: LED, ~, symbol LED
- removed J201: DB9, symbol DB9
- removed R201: R, ~, symbol R
- removed U201: ISL83387E, ~, symbol ISL83387E
Connections:
- net labels removed: A_CTS, A_DSR, A_DTR, A_RTS, A_RX, A_TX, B_CTS, B_DSR, B_DTR, B_RTS
- wire segments 92 -> 46
- no-connect marks 2 -> 8
