File: boards/GPIO-8 daughterboard/PIC-GPIO8.sch (KiCad schematic (older format))
At the start: 9 parts, among them P301 ICSP, U301 PIC16F1704

Commit message: Updated GPIO8 dboard to use RS232 adapter block; Changed power hierarchy pin in RS232_adapter_block and PIC-GPIO8 sheets as passive type
Changed lines of the file:
@@
 $Descr A4 11693 8268
 encoding utf-8
-Sheet 3 3
+Sheet 3 4
 Title ""
 Date "1 jul 2014"
@@
 Comment4 ""
 $EndDescr
-Text HLabel 3900 3300 0    60   Input ~ 0
+Text HLabel 3900 3300 0    60   UnSpc ~ 0
 VCC
-Text HLabel 3900 3700 0    60   Input ~ 0
+Text HLabel 3900 3700 0    60   UnSpc ~ 0
 GND
 Text HLabel 7350 3300 2    60   BiDi ~ 0
@@
 Wire Wire Line
 	7400 5150 7500 5150
-Text HLabel 7500 5150 2    60   Input ~ 0
+Text HLabel 7500 5150 2    60   UnSpc ~ 0
 GND
 Wire Wire Line
