File: boards/RS232C daughterboard/RS232C standalone.sch (KiCad schematic (older format))
At the start: 2 parts

Commit message: Completed RS232C daughterboard
Parts:
- added C? (x12): 0.1u, ~, symbol CSMALL
- added D? (x2): LED, ~, symbol LED
- added J? (x2): DB9, symbol DB9
- added R? (x2): R, ~, symbol R
- added U?: ISL83387E, ~, symbol ISL83387E
Connections:
- net labels added: A_CTS, A_DSR, A_DTR, A_GND, A_RTS, A_RX, A_TX, B_CTS, B_DSR, B_DTR, B_RTS, B_RX, B_TX, C_CTS, C_DSR, C_DTR, C_GND, C_RTS, C_RX, C_TX
- wire segments 11 -> 138
- no-connect marks 0 -> 4
Other:
- note added: "DTE Serial DB9 pinout:\n1 DCD <-- Data Carrier Detect\n2 RXD <-- Receive Data\n3 TXD --> Transmit Data\n4 DTR --> Data Terminal Ready\n5 GND --- System Ground\n6 DSR <-- Data Set Ready\n7 RTS --> Request to Send\n8 CTS <-- Clear to Send\n9 RI <-- Ring Indicator"
- moved on the sheet: U?

Commit message: Fixed errors in RS232C daughterboard, ERC passed
Parts:
- gave numbers to parts that had none: 21
Connections:
- net labels removed: A_GND, C_GND
- wire segments 138 -> 129
Changed lines of the file:
@@
 A0
 $Comp
-L 24AA014 U?
+L 24AA014 U202
 U 1 1 53ABBAB7
 P 5500 6650
-F 0 "U?" H 5650 7000 60  0000 C CNN
+F 0 "U202" H 5650 7000 60  0000 C CNN
 F 1 "24AA014" H 5700 6300 60  0000 C CNN
 F 2 "~" H 5500 6650 60  0000 C CNN
@@
 $EndComp
 $Comp
-L ISL83387E U?
+L ISL83387E U203
 U 1 1 53ABBB03
 P 7650 3350
-F 0 "U?" H 7250 2400 60  0000 L CNN
+F 0 "U203" H 7250 2400 60  0000 L CNN
 F 1 "ISL83387E" H 7250 4250 60  0000 L CNN
 F 2 "~" H 7650 3350 60  0000 C CNN
@@
 $EndComp
 $Comp
-L DB9 J?
+L DB9 J201
 U 1 1 53ABC2C6
 P 1100 3550
-F 0 "J?" H 1100 4100 70  0000 C CNN
+F 0 "J201" H 1100 4100 70  0000 C CNN
 F 1 "DB9" H 1100 3000 70  0000 C CNN
 F 2 "" H 1100 3550 60  0000 C CNN
@@
 $EndComp
 $Comp
-L CSMALL C?
+L CSMALL C212
 U 1 1 53ABC31D
 P 9000 2750
-F 0 "C?" H 9025 2800 30  0000 L CNN
+F 0 "C212" H 9025 2800 30  0000 L CNN
 F 1 "0.1u" H 9025 2700 30  0000 L CNN
 F 2 "~" H 9000 2750 60  0000 C CNN
@@
 $EndComp
 $Comp
-L CSMALL C?
+L CSMALL C211
 U 1 1 53ABC32C
 P 8800 2850
-F 0 "C?" H 8825 2900 30  0000 L CNN
+F 0 "C211" H 8825 2900 30  0000 L CNN
 F 1 "0.1u" H 8825 2800 30  0000 L CNN
 F 2 "~" H 8800 2850 60  0000 C CNN
@@
 $EndComp
 $Comp
-L CSMALL C?
+L CSMALL C210
 U 1 1 53ABC33B
 P 8650 3050
-F 0 "C?" H 8675 3100 30  0000 L CNN
+F 0 "C210" H 8675 3100 30  0000 L CNN
 F 1 "0.1u" H 8675 3000 30  0000 L CNN
 F 2 "~" H 8650 3050 60  0000 C CNN
@@
 $EndComp
 $Comp
-L CSMALL C?
+L CSMALL C209
 U 1 1 53ABC34A
 P 8500 3100
-F 0 "C?" H 8525 3150 30  0000 L CNN
+F 0 "C209" H 8525 3150 30  0000 L CNN
 F 1 "0.1u" H 8525 3050 30  0000 L CNN
 F 2 "~" H 8500 3100 60  0000 C CNN
@@
 $EndComp
 $Comp
-L CSMALL C?
+L CSMALL C207
 U 1 1 53ABC393
 P 6750 2650
-F 0 "C?" H 6775 2700 30  0000 L CNN
+F 0 "C207" H 6775 2700 30  0000 L CNN
 F 1 "0.1u" H 6775 2600 30  0000 L CNN
 F 2 "~" H 6750 2650 60  0000 C CNN
@@
 $EndComp
 $Comp
-L CSMALL C?
+L CSMALL C208
 U 1 1 53ABC399
 P 6750 3000
-F 0 "C?" H 6775 3050 30  0000 L CNN
+F 0 "C208" H 6775 3050 30  0000 L CNN
 F 1 "0.1u" H 6775 2950 30  0000 L CNN
 F 2 "~" H 6750 3000 60  0000 C CNN
@@
 GND_ISO
 $Comp
-L LED D?
+L LED D202
 U 1 1 53ABCB34
 P 6300 4400
-F 0 "D?" H 6300 4500 50  0000 C CNN
+F 0 "D202" H 6300 4500 50  0000 C CNN
 F 1 "LED" H 6300 4300 50  0000 C CNN
 F 2 "~" H 6300 4400 60  0000 C CNN
@@
 $EndComp
 $Comp
-L R R?
+L R R202
 U 1 1 53ABCB43
 P 6600 4150
-F 0 "R?" V 6550 3950 40  0000 C CNN
+F 0 "R202" V 6550 3950 40  0000 C CNN
 F 1 "R" V 6607 4151 40  0000 C CNN
 F 2 "~" V 6530 4150 30  0000 C CNN
@@
 VCC_5V_ISO
 $Comp
-L ISL83387E U?
+L ISL83387E U201
 U 1 1 53ABD102
 P 4100 3350
-F 0 "U?" H 3700 2400 60  0000 L CNN
+F 0 "U201" H 3700 2400 60  0000 L CNN
 F 1 "ISL83387E" H 3700 4250 60  0000 L CNN
 F 2 "~" H 4100 3350 60  0000 C CNN
@@
 $EndComp
 $Comp
-L CSMALL C?
+L CSMALL C201
 U 1 1 53ABD108
 P 2750 2750
-F 0 "C?" H 2775 2800 30  0000 L CNN
+F 0 "C201" H 2775 2800 30  0000 L CNN
 F 1 "0.1u" H 2775 2700 30  0000 L CNN
 F 2 "~" H 2750 2750 60  0000 C CNN
@@
 $EndComp
 $Comp
-L CSMALL C?
+L CSMALL C202
 U 1 1 53ABD10E
 P 2950 2850
-F 0 "C?" H 2975 2900 30  0000 L CNN
+F 0 "C202" H 2975 2900 30  0000 L CNN
 F 1 "0.1u" H 2975 2800 30  0000 L CNN
 F 2 "~" H 2950 2850 60  0000 C CNN
@@
 $EndComp
 $Comp
-L CSMALL C?
+L CSMALL C203
 U 1 1 53ABD114
 P 3100 3050
-F 0 "C?" H 3125 3100 30  0000 L CNN
+F 0 "C203" H 3125 3100 30  0000 L CNN
 F 1 "0.1u" H 3125 3000 30  0000 L CNN
 F 2 "~" H 3100 3050 60  0000 C CNN
@@
 $EndComp
 $Comp
-L CSMALL C?
+L CSMALL C204
 U 1 1 53ABD11A
 P 3250 3100
-F 0 "C?" H 3275 3150 30  0000 L CNN
+F 0 "C204" H 3275 3150 30  0000 L CNN
 F 1 "0.1u" H 3275 3050 30  0000 L CNN
 F 2 "~" H 3250 3100 60  0000 C CNN
@@
 $EndComp
 $Comp
-L CSMALL C?
+L CSMALL C205
 U 1 1 53ABD120
 P 5000 2650
-F 0 "C?" H 5025 2700 30  0000 L CNN
+F 0 "C205" H 5025 2700 30  0000 L CNN
 F 1 "0.1u" H 5025 2600 30  0000 L CNN
 F 2 "~" H 5000 2650 60  0000 C CNN
@@
 $EndComp
 $Comp
-L CSMALL C?
+L CSMALL C206
 U 1 1 53ABD126
 P 5000 3000
-F 0 "C?" H 5025 3050 30  0000 L CNN
+F 0 "C206" H 5025 3050 30  0000 L CNN
 F 1 "0.1u" H 5025 2950 30  0000 L CNN
 F 2 "~" H 5000 3000 60  0000 C CNN
@@
 GND_ISO
 $Comp
-L LED D?
+L LED D201
 U 1 1 53ABD150
 P 5450 4400
-F 0 "D?" H 5450 4500 50  0000 C CNN
+F 0 "D201" H 5450 4500 50  0000 C CNN
 F 1 "LED" H 5450 4300 50  0000 C CNN
 F 2 "~" H 5450 4400 60  0000 C CNN
@@
 $EndComp
 $Comp
-L R R?
+L R R201
 U 1 1 53ABD156
 P 5150 4150
-F 0 "R?" V 5100 3950 40  0000 C CNN
+F 0 "R201" V 5100 3950 40  0000 C CNN
 F 1 "R" V 5157 4151 40  0000 C CNN
 F 2 "~" V 5080 4150 30  0000 C CNN
@@
 Text Notes 1050 6450 0    60   ~ 0
 DTE Serial DB9 pinout:\n1	DCD	<--	Data Carrier Detect\n2	RXD	<--	Receive Data\n3	TXD	-->	Transmit Data\n4	DTR	-->	Data Terminal Ready\n5	GND	---	System Ground\n6	DSR	<--	Data Set Ready\n7	RTS	-->	Request to Send\n8	CTS	<--	Clear to Send\n9	RI	<--	Ring Indicator
-Text Label 1700 3150 0    60   ~ 0
-A_GND
 Text Label 1700 3350 0    60   ~ 0
 A_DTR
@@
 Text Label 2550 3650 2    60   ~ 0
 A_DSR
-Text Label 10100 3050 2    60   ~ 0
-C_GND
 Text Label 10100 3250 2    60   ~ 0
 C_DTR
@@
 NoConn ~ 10250 3150
 $Comp
-L DB9 J?
+L DB9 J202
 U 1 1 53ABD89D
 P 10700 3450
-F 0 "J?" H 10700 4000 70  0000 C CNN
+F 0 "J202" H 10700 4000 70  0000 C CNN
 F 1 "DB9" H 10700 2900 70  0000 C CNN
 F 2 "" H 10700 3450 60  0000 C CNN
@@
 	4700 6850 4700 7200
 Wire Wire Line
-	4550 7200 4700 7200
-Wire Wire Line
-	4700 7200 5500 7200
+	4550 7200 5500 7200
 Wire Wire Line
 	5500 7200 5500 7150
@@
 	9000 2600 9000 2650
 Wire Wire Line
-	8800 2350 8800 2600
-Wire Wire Line
-	8800 2600 8800 2700
-Wire Wire Line
-	8800 2700 8800 2750
+	8800 2350 8800 2750
 Connection ~ 8800 2700
 Wire Wire Line
-	8350 4150 8500 4150
-Wire Wire Line
-	8500 4150 8650 4150
-Wire Wire Line
-	8650 4150 8800 4150
-Wire Wire Line
-	8800 4150 9000 4150
-Wire Wire Line
-	9000 4150 9100 4150
+	8350 4150 9100 4150
 Wire Wire Line
 	8800 2950 8800 4150
@@
 	6300 4650 6300 4600
 Wire Wire Line
-	8350 2600 8800 2600
-Wire Wire Line
-	8800 2600 9000 2600
+	8350 2600 9000 2600
 Wire Wire Line
 	8500 2900 8350 2900
@@
 	2750 2650 2750 2600
 Wire Wire Line
-	2950 2350 2950 2600
-Wire Wire Line
-	2950 2600 2950 2700
-Wire Wire Line
-	2950 2700 2950 2750
+	2950 2350 2950 2750
 Connection ~ 2950 2700
 Wire Wire Line
-	2650 4150 2750 4150
-Wire Wire Line
-	2750 4150 2950 4150
-Wire Wire Line
-	2950 4150 3100 4150
-Wire Wire Line
-	3100 4150 3250 4150
-Wire Wire Line
-	3250 4150 3400 4150
+	2650 4150 3400 4150
 Wire Wire Line
 	2950 2950 2950 4150
@@
 	5450 4650 5450 4600
 Wire Wire Line
-	2750 2600 2950 2600
-Wire Wire Line
-	2950 2600 3400 2600
+	2750 2600 3400 2600
 Wire Wire Line
 	3250 2900 3400 2900
@@
 	10250 3650 10100 3650
 Wire Wire Line
+	10250 3250 10100 3250
+Wire Wire Line
+	10250 3350 10100 3350
+Wire Wire Line
+	10250 3750 10100 3750
+Wire Wire Line
+	10250 3450 10100 3450
+Wire Wire Line
+	10250 3550 10100 3550
+$Comp
+L PWR_FLAG #FLG01
+U 1 1 53ABE834
+P 2950 2350
+F 0 "#FLG01" H 2950 2445 30  0001 C CNN
+F 1 "PWR_FLAG" H 2950 2530 30  0001 C CNN
+F 2 "" H 2950 2350 60  0000 C CNN
+F 3 "" H 2950 2350 60  0000 C CNN
+	1    2950 2350
+	1    0    0    -1
+$EndComp
+$Comp
+L PWR_FLAG #FLG02
+U 1 1 53ABE907
+P 5500 6050
+F 0 "#FLG02" H 5500 6145 30  0001 C CNN
+F 1 "PWR_FLAG" H 5500 6230 30  0001 C CNN
+F 2 "" H 5500 6050 60  0000 C CNN
+F 3 "" H 5500 6050 60  0000 C CNN
+	1    5500 6050
+	1    0    0    -1
+$EndComp
+$Comp
+L PWR_FLAG #FLG03
+U 1 1 53ABE910
+P 7050 6050
+F 0 "#FLG03" H 7050 6145 30  0001 C CNN
+F 1 "PWR_FLAG" H 7050 6230 30  0001 C CNN
+F 2 "" H 7050 6050 60  0000 C CNN
+F 3 "" H 7050 6050 60  0000 C CNN
+	1    7050 6050
+	1    0    0    -1
+$EndComp
+$Comp
+L PWR_FLAG #FLG04
+U 1 1 53ABE916
+P 7050 6550
+F 0 "#FLG04" H 7050 6645 30  0001 C CNN
+F 1 "PWR_FLAG" H 7050 6730 30  0001 C CNN
+F 2 "" H 7050 6550 60  0000 C CNN
+F 3 "" H 7050 6550 60  0000 C CNN
+	1    7050 6550
+	1    0    0    -1
+$EndComp
+Wire Wire Line
+	7050 6050 7050 6200
+Wire Wire Line
+	7050 6200 7250 6200
+Wire Wire Line
+	7050 6550 7050 6700
+Wire Wire Line
+	7050 6700 7250 6700
+Text HLabel 7250 6200 2    60   Input ~ 0
+GND
+Text HLabel 7250 6700 2    60   Input ~ 0
+GND_ISO
+Text HLabel 1700 3000 1    60   Input ~ 0
+GND_ISO
+Wire Wire Line
+	1700 3150 1700 3000
+Wire Wire Line
 	10250 3050 10100 3050
-Wire Wire Line
-	10250 3250 10100 3250
-Wire Wire Line
-	10250 3350 10100 3350
-Wire Wire Line
-	10250 3750 10100 3750
-Wire Wire Line
-	10250 3450 10100 3450
-Wire Wire Line
-	10250 3550 10100 3550
+Text HLabel 10100 2900 1    60   Input ~ 0
+GND_ISO
+Wire Wire Line
+	10100 3050 10100 2900
 $EndSCHEMATC

Commit message: Added currentlimiting resistor to RS232 dboard eeprom
Parts:
- added R203: 50, ~, symbol R
Connections:
- wire segments 129 -> 130
Changed lines of the file:
@@
 Text HLabel 5600 2350 1    60   Output ~ 0
 DSR_ISO
-Text HLabel 5400 6050 0    60   Input ~ 0
+Text HLabel 4700 6050 0    60   Input ~ 0
 VCC_3V3
 Text HLabel 4550 7200 0    60   Input ~ 0
@@
 	6300 6550 6200 6550
 Wire Wire Line
-	5400 6050 5500 6050
+	5300 6050 5500 6050
 Wire Wire Line
 	5500 6050 5500 6150
@@
 	10250 3550 10100 3550
 $Comp
-L PWR_FLAG #FLG01
+L PWR_FLAG #FLG201
 U 1 1 53ABE834
 P 2950 2350
-F 0 "#FLG01" H 2950 2445 30  0001 C CNN
+F 0 "#FLG201" H 2950 2445 30  0001 C CNN
 F 1 "PWR_FLAG" H 2950 2530 30  0001 C CNN
 F 2 "" H 2950 2350 60  0000 C CNN
@@
 $EndComp
 $Comp
-L PWR_FLAG #FLG02
+L PWR_FLAG #FLG202
 U 1 1 53ABE907
 P 5500 6050
-F 0 "#FLG02" H 5500 6145 30  0001 C CNN
+F 0 "#FLG202" H 5500 6145 30  0001 C CNN
 F 1 "PWR_FLAG" H 5500 6230 30  0001 C CNN
 F 2 "" H 5500 6050 60  0000 C CNN
@@
 $EndComp
 $Comp
-L PWR_FLAG #FLG03
+L PWR_FLAG #FLG203
 U 1 1 53ABE910
 P 7050 6050
-F 0 "#FLG03" H 7050 6145 30  0001 C CNN
+F 0 "#FLG203" H 7050 6145 30  0001 C CNN
 F 1 "PWR_FLAG" H 7050 6230 30  0001 C CNN
 F 2 "" H 7050 6050 60  0000 C CNN
@@
 $EndComp
 $Comp
-L PWR_FLAG #FLG04
+L PWR_FLAG #FLG204
 U 1 1 53ABE916
 P 7050 6550
-F 0 "#FLG04" H 7050 6645 30  0001 C CNN
+F 0 "#FLG204" H 7050 6645 30  0001 C CNN
 F 1 "PWR_FLAG" H 7050 6730 30  0001 C CNN
 F 2 "" H 7050 6550 60  0000 C CNN
@@
 Wire Wire Line
 	10100 3050 10100 2900
+$Comp
+L R R203
+U 1 1 53ABAC25
+P 5050 6050
+F 0 "R203" V 5130 6050 40  0000 C CNN
+F 1 "50" V 5057 6051 40  0000 C CNN
+F 2 "~" V 4980 6050 30  0000 C CNN
+F 3 "~" H 5050 6050 30  0000 C CNN
+	1    5050 6050
+	0    -1   -1   0
+$EndComp
+Wire Wire Line
+	4800 6050 4700 6050
 $EndSCHEMATC

Commit message: Removed RS232 adapter input module from RS232C daughterboard
Parts:
- removed C201, C202, C203, C204, C205, C206: 0.1u, ~, symbol CSMALL
- removed D201: LED, ~, symbol LED
- removed J201: DB9, symbol DB9
- removed R201: R, ~, symbol R
- removed U201: ISL83387E, ~, symbol ISL83387E
Connections:
- net labels removed: A_CTS, A_DSR, A_DTR, A_RTS, A_RX, A_TX, B_CTS, B_DSR, B_DTR, B_RTS, B_RX, B_TX
- wire segments 130 -> 70
- no-connect marks 4 -> 2
Other:
- moved on the sheet: D202, J202, R202, U203

Commit message: Reviewed RS232C schematics; Updated R202; Changed power hierarchical pins to passive
Parts:
- R202: value R -> 1.5K
Changed lines of the file:
@@
 Sheet 2 2
 Title ""
-Date "2 jul 2014"
+Date "3 jul 2014"
 Rev ""
 Comp ""
@@
 Text HLabel 3700 3550 0    60   Output ~ 0
 DSR_ISO
-Text HLabel 4700 6050 0    60   Input ~ 0
+Text HLabel 4700 6050 0    60   UnSpc ~ 0
 VCC_3V3
-Text HLabel 4550 7200 0    60   Input ~ 0
+Text HLabel 4550 7200 0    60   UnSpc ~ 0
 GND
 Text HLabel 6050 2150 0    60   Input ~ 0
@@
 	-1   0    0    -1
 $EndComp
-Text HLabel 6500 3950 2    60   Input ~ 0
-GND_ISO
-Text HLabel 4250 3850 0    60   Input ~ 0
+Text HLabel 6500 3950 2    60   UnSpc ~ 0
+GND_ISO
+Text HLabel 4250 3850 0    60   UnSpc ~ 0
 VCC_5V_ISO
-Text HLabel 4250 3750 0    60   Input ~ 0
+Text HLabel 4250 3750 0    60   UnSpc ~ 0
 GND_ISO
 $Comp
@@
 U 1 1 53ABCB43
 P 4000 3950
-F 0 "R202" V 3950 3750 40  0000 C CNN
-F 1 "R" V 4007 3951 40  0000 C CNN
+F 0 "R202" V 3950 3700 40  0000 C CNN
+F 1 "1.5K" V 4007 3951 40  0000 C CNN
 F 2 "~" V 3930 3950 30  0000 C CNN
 F 3 "~" H 4000 3950 30  0000 C CNN
@@
 	0    -1   -1   0
 $EndComp
-Text HLabel 3750 4450 2    60   Input ~ 0
+Text HLabel 3750 4450 2    60   UnSpc ~ 0
 GND_ISO
 Text Notes 1050 6450 0    60   ~ 0
@@
 Wire Wire Line
 	7050 6700 7250 6700
-Text HLabel 7250 6200 2    60   Input ~ 0
+Text HLabel 7250 6200 2    60   UnSpc ~ 0
 GND
-Text HLabel 7250 6700 2    60   Input ~ 0
+Text HLabel 7250 6700 2    60   UnSpc ~ 0
 GND_ISO
 Wire Wire Line
 	7650 2850 7500 2850
-Text HLabel 7500 2700 1    60   Input ~ 0
-GND_ISO
-Wire Wire Line
+Text HLabel 7500 2700 1    60   UnSpc ~ 0
+GND_ISO
+Wire Wire Line

Commit message: Added bypass capacitor to EEPROM in RS232C dboard
Parts:
- added C201: 0.1u, ~, symbol CSMALL
Connections:
- wire segments 70 -> 73
Other:
- moved on the sheet: R203
Changed lines of the file:
@@
 Text HLabel 3700 3550 0    60   Output ~ 0
 DSR_ISO
-Text HLabel 4700 6050 0    60   UnSpc ~ 0
+Text HLabel 4300 6050 0    60   UnSpc ~ 0
 VCC_3V3
 Text HLabel 4550 7200 0    60   UnSpc ~ 0
@@
 	6300 6550 6200 6550
 Wire Wire Line
-	5300 6050 5500 6050
+	4900 6050 5500 6050
 Wire Wire Line
 	5500 6050 5500 6150
@@
 L R R203
 U 1 1 53ABAC25
-P 5050 6050
-F 0 "R203" V 5130 6050 40  0000 C CNN
-F 1 "50" V 5057 6051 40  0000 C CNN
-F 2 "~" V 4980 6050 30  0000 C CNN
-F 3 "~" H 5050 6050 30  0000 C CNN
-	1    5050 6050
+P 4650 6050
+F 0 "R203" V 4730 6050 40  0000 C CNN
+F 1 "50" V 4657 6051 40  0000 C CNN
+F 2 "~" V 4580 6050 30  0000 C CNN
+F 3 "~" H 4650 6050 30  0000 C CNN
+	1    4650 6050
 	0    -1   -1   0
 $EndComp
 Wire Wire Line
-	4800 6050 4700 6050
+	4400 6050 4300 6050
 $Comp
 L PWR_FLAG #FLG04
@@
 $EndComp
 Connection ~ 6200 2150
+$Comp
+L CSMALL C201
+U 1 1 53B5143E
+P 5150 5850
+F 0 "C201" H 5175 5900 30  0000 L CNN
+F 1 "0.1u" H 5175 5800 30  0000 L CNN
+F 2 "~" H 5150 5850 60  0000 C CNN
+F 3 "~" H 5150 5850 60  0000 C CNN
+	1    5150 5850
+	1    0    0    -1
+$EndComp
+Wire Wire Line
+	5150 5950 5150 6050
+Connection ~ 5150 6050
+Wire Wire Line
+	5150 5650 5150 5750
+Wire Wire Line
+	4750 5650 5150 5650
+Text HLabel 4750 5650 0    60   UnSpc ~ 0
+GND
 $EndSCHEMATC
