File: boards/RS232C daughterboard/RS232C standalone.sch (KiCad schematic (older format))
At the start: 13 parts, among them J202 DB9, U202 24AA014, U203 ISL83387E

Commit message: Changed LED resistor in RS232C dboard to 820R to be 3.3-5V compatible
Parts:
- R202: value 1.5K -> 820
Changed lines of the file:
@@
 P 4000 3950
 F 0 "R202" V 3950 3700 40  0000 C CNN
-F 1 "1.5K" V 4007 3951 40  0000 C CNN
+F 1 "820" V 4007 3951 40  0000 C CNN
 F 2 "~" V 3930 3950 30  0000 C CNN
 F 3 "~" H 4000 3950 30  0000 C CNN
