File: boards/MIDI daughterboard/MIDI standalone.sch (KiCad schematic (older format))
At the start: 13 parts, among them J201 DB9, J202 DB9, U201 ISL83387E, U202 24AA014

Commit message: Added bypass capacitor to EEPROM in MIDI dboard template and cleaned template
Parts:
- removed C202, C203, C204, C205, C206: 0.1u, ~, symbol CSMALL
- removed D201: LED, ~, symbol LED
- removed J201, J202: DB9, symbol DB9
- removed R201: R, ~, symbol R
- removed U201: ISL83387E, ~, symbol ISL83387E
Connections:
- net labels removed: A_CTS, A_DSR, A_DTR, A_RTS, A_RX, A_TX, B_CTS, B_DSR, B_DTR, B_RTS, B_RX, B_TX, CTS_ISO, C_CTS, C_DSR, C_DTR, C_RTS, C_RX, C_TX, DSR_ISO, DTR_ISO, RTS_ISO, RX_ISO, TX_ISO, VCC_5V_ISO
- wire segments 90 -> 19
- no-connect marks 4 -> 0
Other:
- note removed: "DTE Serial DB9 pinout:\n1 DCD <-- Data Carrier Detect\n2 RXD <-- Receive Data\n3 TXD --> Transmit Data\n4 DTR --> Data Terminal Ready\n5 GND --- System Ground\n6 DSR <-- Data Set Ready\n7 RTS --> Request to Send\n8 CTS <-- Clear to Send\n9 RI <-- Ring Indicator"
- moved on the sheet: R203

Commit message: Done MIDI daughterboard; Changed bypass capacitor in RS232_adapter_block from 0.1u to 1.0u
Parts:
- added D201: 1N914, ~, symbol DIODE
- added IC201: 6N138, DIP8, symbol 6N136
- added P201: MIDI_IN, ~, symbol DIN_5_MODIFIED
- added P202: MIDI_OUT, ~, symbol DIN_5_MODIFIED
- added R201: 1k, ~, symbol R
- added R202, R204: 220, ~, symbol R
Connections:
- net labels added: CTS_ISO, DSR_ISO, DTR_ISO, RTS_ISO, RX_ISO, TX_ISO, VCC_5V_ISO
- wire segments 19 -> 55
- no-connect marks 0 -> 14
Other:
- moved on the sheet: R203, U202
