File: boards/LED daughterboard/LED standalone.sch (KiCad schematic (older format))
At the start: 13 parts, among them J201 DB9, J202 DB9, U201 ISL83387E, U202 24AA014

Commit message: Added bypass capacitor to EEPROM in LED dboard and cleaned template
Parts:
- removed C202, C203, C204, C205, C206: 0.1u, ~, symbol CSMALL
- removed D201: LED, ~, symbol LED
- removed J201, J202: DB9, symbol DB9
- removed R201: R, ~, symbol R
- removed U201: ISL83387E, ~, symbol ISL83387E
Connections:
- net labels removed: A_CTS, A_DSR, A_DTR, A_RTS, A_RX, A_TX, B_CTS, B_DSR, B_DTR, B_RTS, B_RX, B_TX, CTS_ISO, C_CTS, C_DSR, C_DTR, C_RTS, C_RX, C_TX, DSR_ISO, DTR_ISO, RTS_ISO, RX_ISO, TX_ISO, VCC_5V_ISO
- wire segments 90 -> 19
- no-connect marks 4 -> 0
Other:
- moved on the sheet: R203
